File: PCB/CertStack/CertStack.brd (EAGLE design)
At the start: 45 x 100 mm, 42 parts, among them J1 MEM2075-00-140-01-A, Q1 AOD4184A, Q2 AOD4184A, Q3 AOD4184A, Q4 AOD4184A, Q5 MMBT2222A, T1 DMP3098L-7, U2 INVENSENSE_ICM-20608-GINVENSE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, U3 SST26VF064B-104V/MN, U4 LT1374CS8-5PBF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

Commit message: PCB
Parts:
- removed XT1: XT30-RH, mylibrary:XT30-RH
- added BATTERY, SWITCH: (no value), pinhead:1X02
- added CAN, I2C: (no value), pinhead:1X04
- added GPS, POWER, SPI, TELEM, VTX: (no value), pinhead:1X06
- renumbered JP1 to CAMERA
Connections:
- net GND: now also BATTERY.2; no longer XT1.-
- net VCC: now also BATTERY.1; no longer XT1.+

Commit message: PCB
Parts:
- removed R21: 360k, rcl:R0805
- removed R22: 51k, rcl:R0805
- removed R23, R5, R6, R9: 10k, rcl:R0805
- removed X1, X2, X3, X4: TERMINAL-BLOCK-3.5MM-2-PIN-LONG-PAD, Rembrandt Electronics - Terminal Block 3-5mm v1-0:TERMINAL-BLOCK-2-PIN-3.5MM-LONG-PAD
- added R1, R2: 10k, rcl:R0805
- Q1, Q2, Q3, Q4: value AOD4184A -> SI2302; device AOD4184A:DPAK228P994X240-4N -> SI2302:SOT23
- R3: value 360k -> 10k
- R4: value 51k -> 10k
- moved POWER 130.1 mm to (34.0, 28.0)
- moved SPI 124.2 mm to (34.0, 23.0)
- moved I2C 123.5 mm to (36.0, 18.0)
- moved CAN 107.7 mm to (24.0, 18.0)
- moved CAMERA 107.6 mm to (10.1, 17.9)
- moved R4 100.7 mm to (-15.0, 16.0)
- moved TELEM 99.0 mm to (13.0, 33.0)
- moved GPS 92.1 mm to (13.0, 23.0)
- moved VTX 91.8 mm to (13.0, 28.0)
- moved Q1 81.8 mm to (-14.0, 62.0)
- moved R3 74.3 mm to (-15.0, 29.0)
- moved C8 66.0 mm to (-16.0, 71.6)
- moved R14 35.7 mm to (37.0, 61.0), turned to 180 degrees
- moved Q4 33.2 mm to (-14.0, 23.0)
- moved BATTERY 31.8 mm to (39.0, 33.0)
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Connections:
- removed net CE: U3.1
- removed net PY1_D: R21.1, R22.2
- removed net PY1_F: Q3.1, R23.2
- removed net PY2_D: R3.1, R4.2
- removed net PY2_F: Q1.1, R5.2
- removed net PY3_F: Q2.1, R6.2
- removed net PY4_F: Q4.1, R9.2
- removed net SDI: BMP384_1.4, U2.3
- removed net SDO: BMP384_1.5, U2.4
- new net BATV: R14.2
- new net CS_FLASH: U$1.2, U3.1
- new net N$1: Q1.1, R1.2
- new net N$10: Q4.1, R4.2
- new net N$11: Q4.3
- new net N$8: Q3.1, R3.2
- net +3V3: no longer BMP384_1.3, C2.2
- net +5V: no longer X2.1, X4.1
- net CS_BAR: now also U$1.6
- net GND: now also BMP384_1.3, C2.2, Q1.2, Q2.2, Q3.2, Q4.2, R1.1, R2.1, R3.1; no longer Q1.3, Q2.3, Q3.3, Q4.3, R22.1, R23.1, R5.1, R6.1, R9.1
- net MISO: now also BMP384_1.5, U2.4
- net MOSI: now also BMP384_1.4, U2.3
- net N$3: now also Q1.3; no longer Q1.4, R3.2, X1.2
- net N$4: now also Q2.1, R2.2; no longer Q4.4, X4.2
- net N$5: now also Q2.3; no longer Q2.4, X2.2
- net N$9: now also Q3.3; no longer Q3.4, R21.2, X3.2
- net VCC: no longer X1.1, X3.1
Routing:
- net SCK: track 0.00 -> 75.7 mm, vias 0 -> 3
- net MOSI: track 0.00 -> 69.0 mm, vias 0 -> 2
- net MISO: track 0.00 -> 46.0 mm, vias 0 -> 2
- net VBUS: track 0.00 -> 45.9 mm
- net +3V3: track 13.6 -> 53.8 mm, vias 0 -> 4
- net CS_BAR: track 0.00 -> 10.2 mm, vias 0 -> 1
- net CS_FLASH: track 0.00 -> 9.47 mm, vias 0 -> 1
- net GND: track 0.00 -> 5.90 mm
- net N$12: track 0.00 -> 3.09 mm

Commit message: PCB
Parts:
- moved R4 50.2 mm to (28.0, 42.0)
- moved Q4 48.4 mm to (28.0, 47.0)
- moved C8 43.6 mm to (22.7, 51.6), turned to 180 degrees
- moved R3 41.1 mm to (24.0, 42.0)
- moved Q3 39.6 mm to (24.0, 47.0)
- moved Q2 34.2 mm to (19.0, 40.0)
- moved R2 34.1 mm to (19.0, 44.0)
- moved Q1 33.2 mm to (10.0, 39.0), turned to 180 degrees
- moved R1 33.1 mm to (14.0, 39.0), turned to 90 degrees

Commit message: PCB
Parts:
- removed CAN, I2C: (no value), pinhead:1X04
- removed SPI: (no value), pinhead:1X06
- removed SWITCH: (no value), pinhead:1X02
- added DATA: (no value), mylibrary:JST-PH-6
- CAMERA: device pinhead:1X04 -> mylibrary:JST-PH-6
- GPS, POWER, TELEM, VTX: device pinhead:1X06 -> mylibrary:JST-PH-6
- moved GPS 20.4 mm to (32.5, 17.0)
- moved CAMERA 11.1 mm to (12.5, 7.00)
- moved VTX 11.0 mm to (12.5, 17.0)
- moved TELEM 6.02 mm to (12.5, 27.0)
- moved POWER 1.80 mm to (32.5, 27.0)
Connections:
- net N$11 renamed FET4
- net N$5 renamed FET3
- removed net VID-IN: CAMERA.3
- new net CANH: DATA.6
- new net CANL: DATA.5
- new net FET1: Q1.3, TELEM.1
- new net FET2: CAMERA.1, Q3.3, VTX.1
- new net GPS_RX: GPS.3
- new net GPS_TX: GPS.4
- new net N$11: GPS.6
- new net SW+: POWER.5
- new net SW-: POWER.6
- new net TELEM_RX: TELEM.3
- new net TELEM_TX: TELEM.4
- new net VIDEO: CAMERA.3, VTX.3
- new net VTX_RX: VTX.4
- new net VTX_TX: VTX.5
- net +3V3: now also DATA.2, GPS.2, POWER.2
- net +5V: now also POWER.3, TELEM.2
- net BATV: now also CAMERA.2, POWER.4, VTX.2
- net GND: now also DATA.1, GPS.1, POWER.1, TELEM.6, VTX.6; no longer CAMERA.2
- net N$2: now also CAMERA.5; no longer CAMERA.1
- net N$3: now also CAMERA.6; no longer Q1.3
- net N$9: now also GPS.5; no longer Q3.3
- net SCL: now also DATA.3
- net SDA: now also DATA.4
Routing:
- net VIDEO: track 0.00 -> 10.0 mm
- net BATV: track 0.00 -> 10.0 mm

Commit message: PCB
Parts:
- moved U4 14.3 mm to (51.9, 48.6)
- moved Q3 13.5 mm to (15.0, 37.0), turned to 180 degrees
- moved Q4 12.8 mm to (20.0, 37.0), turned to 180 degrees
- moved Q2 9.49 mm to (10.0, 37.0), turned to 180 degrees
- moved R2 9.49 mm to (10.0, 41.0)
- moved R1 9.22 mm to (5.00, 41.0), turned to 0 degrees
- moved R3 9.06 mm to (15.0, 41.0)
- moved C2 8.73 mm to (3.50, 77.0), turned to 270 degrees
- moved R4 8.06 mm to (20.0, 41.0)
- moved Q1 5.39 mm to (5.00, 37.0)
- moved BMP384_1 4.00 mm to (7.00, 77.0), turned to 90 degrees
- moved C1 3.50 mm to (10.5, 77.0), turned to 270 degrees
- moved BATTERY 3.00 mm to (39.0, 36.0)
- moved CAMERA 2.00 mm to (12.5, 9.00)
- moved DATA 2.00 mm to (32.5, 9.00)
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Connections:
- removed net N$1: Q1.1, R1.2
- removed net N$10: Q4.1, R4.2
- removed net N$4: Q2.1, R2.2
- removed net N$8: Q3.1, R3.2
- new net F1_TRIG: Q1.1, R1.2, U$1.3
- new net F2_TRIG: Q2.1, R2.2, U$1.4
- new net F3_TRIG: Q3.1, R3.2, U$1.5
- new net F4_TRIG: Q4.1, R4.2, U$1.6
- net CS_BAR: no longer U$1.6
- net FET2: now also Q2.3; no longer Q3.3
- net FET3: now also Q3.3; no longer Q2.3
- net GPS_RX: now also U$1.9
- net GPS_TX: now also U$1.10
- net TELEM_RX: now also U$1.0
- net TELEM_TX: now also U$1.1
- net VTX_RX: now also U$1.7
- net VTX_TX: now also U$1.8
Routing:
- net TELEM_RX: track 0.00 -> 87.4 mm, vias 0 -> 1
- net TELEM_TX: track 0.00 -> 87.1 mm, vias 0 -> 1
- net VTX_RX: track 0.00 -> 84.9 mm, vias 0 -> 1
- net VTX_TX: track 0.00 -> 79.6 mm, vias 0 -> 1
- net F4_TRIG: track 0.00 -> 68.1 mm, vias 0 -> 1
- net F3_TRIG: track 0.00 -> 65.5 mm, vias 0 -> 1
- net F2_TRIG: track 0.00 -> 64.3 mm, vias 0 -> 1
- net F1_TRIG: track 0.00 -> 63.2 mm, vias 0 -> 1
- net FET2: track 0.00 -> 27.9 mm, vias 0 -> 2
- net +5V: track 0.00 -> 20.8 mm, vias 0 -> 1
- net MISO: track 46.0 -> 56.7 mm, vias 2 -> 3
- net CS_BAR: track 10.2 -> 1.17 mm
- net +3V3: track 53.8 -> 62.3 mm, vias 4 -> 2
- net FET1: track 0.00 -> 7.94 mm
- net MOSI: track 69.0 -> 65.1 mm
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
Commit message: PCB
Routing:
- net GPS_TX: track 0.00 -> 93.0 mm, vias 0 -> 1
- net GPS_RX: track 0.00 -> 92.8 mm, vias 0 -> 1
Changed lines of the file:
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@@
 <contactref element="GPS" pad="3"/>
 <contactref element="U$1" pad="9"/>
-<wire x1="31.5" y1="19" x2="14.88" y2="72.22" width="0" layer="19" extent="1-1"/>
+<via x="31.5" y="22.5" extent="1-16" drill="0.35"/>
+<wire x1="31.5" y1="19" x2="31.5" y2="22.5" width="0.5" layer="1"/>
+<wire x1="31.5" y1="22.5" x2="31.5" y2="24.5" width="0.2" layer="15"/>
+<wire x1="31.5" y1="24.5" x2="30.2" y2="25.8" width="0.2" layer="15"/>
+<wire x1="30.2" y1="25.8" x2="3.2" y2="25.8" width="0.2" layer="15"/>
+<wire x1="3.2" y1="25.8" x2="2.4" y2="26.6" width="0.2" layer="15"/>
+<wire x1="2.4" y1="26.6" x2="2.4" y2="70.9" width="0.2" layer="15"/>
+<wire x1="2.4" y1="70.9" x2="3.72" y2="72.22" width="0.2" layer="15"/>
+<wire x1="3.72" y1="72.22" x2="14.88" y2="72.22" width="0.2" layer="15"/>
 </signal>
 <signal name="GPS_TX">
 <contactref element="GPS" pad="4"/>
 <contactref element="U$1" pad="10"/>
-<wire x1="33.5" y1="19" x2="14.88" y2="69.68" width="0" layer="19" extent="1-1"/>
+<via x="33.5" y="22.5" extent="1-16" drill="0.35"/>
+<wire x1="33.5" y1="19" x2="33.5" y2="22.5" width="0.5" layer="1"/>
+<wire x1="33.5" y1="22.5" x2="33.5" y2="24.9" width="0.2" layer="15"/>
+<wire x1="33.5" y1="24.9" x2="31.8" y2="26.6" width="0.2" layer="15"/>
+<wire x1="31.8" y1="26.6" x2="4" y2="26.6" width="0.2" layer="15"/>
+<wire x1="4" y1="26.6" x2="3" y2="27.6" width="0.2" layer="15"/>
+<wire x1="3" y1="27.6" x2="3" y2="70" width="0.2" layer="15"/>
+<wire x1="3" y1="70" x2="4.3" y2="71.3" width="0.2" layer="15"/>
+<wire x1="13.26" y1="71.3" x2="14.88" y2="69.68" width="0.2" layer="15"/>
+<wire x1="4.3" y1="71.3" x2="13.26" y2="71.3" width="0.2" layer="15"/>
 </signal>
 <signal name="N$9">

Commit message: PCB
Routing:
- net +3V3: track 62.3 -> 68.0 mm, vias 2 -> 4
- net VTX_RX: track 84.9 -> 80.6 mm
Changed lines of the file:
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@@
 <wire x1="8.2" y1="88.5" x2="6.4" y2="90.3" width="0.3" layer="16"/>
 <wire x1="6.4" y1="90.3" x2="6.4" y2="93.2" width="0.3" layer="16"/>
-<wire x1="6.215" y1="77.225" x2="5.49" y2="77.95" width="0.2" layer="1"/>
-<wire x1="5.49" y1="77.95" x2="3.5" y2="77.95" width="0.2" layer="1"/>
-<wire x1="10.5" y1="77.95" x2="9.45" y2="79" width="0.2" layer="1"/>
-<wire x1="9.45" y1="79" x2="7" y2="79" width="0.2" layer="1"/>
-<wire x1="7" y1="79" x2="6.55" y2="78.55" width="0.2" layer="1"/>
-<wire x1="6.55" y1="78.55" x2="6.55" y2="77.785" width="0.2" layer="1"/>
+<wire x1="6.215" y1="77.225" x2="5.54" y2="77.9" width="0.2" layer="1"/>
+<wire x1="10.5" y1="77.95" x2="9.95" y2="78.5" width="0.2" layer="1"/>
+<wire x1="9.95" y1="78.5" x2="6.8" y2="78.5" width="0.2" layer="1"/>
+<wire x1="6.8" y1="78.5" x2="6.55" y2="78.25" width="0.2" layer="1"/>
+<wire x1="6.55" y1="78.25" x2="6.55" y2="77.785" width="0.2" layer="1"/>
+<via x="8.2" y="80" extent="1-16" drill="0.35"/>
+<wire x1="8.2" y1="80" x2="8.2" y2="81.75" width="0.3" layer="1"/>
+<wire x1="8.2" y1="81.75" x2="7.95" y2="82" width="0.3" layer="1"/>
+<via x="4.9" y="77.9" extent="1-16" drill="0.35"/>
+<wire x1="4.9" y1="77.9" x2="5.54" y2="77.9" width="0.2" layer="1"/>
+<wire x1="4.9" y1="77.9" x2="3.55" y2="77.9" width="0.2" layer="1"/>
+<wire x1="3.55" y1="77.9" x2="3.5" y2="77.95" width="0.2" layer="1"/>
+<wire x1="4.9" y1="77.9" x2="7" y2="80" width="0.2" layer="16"/>
+<wire x1="7" y1="80" x2="8.2" y2="80" width="0.2" layer="16"/>
 <wire x1="11" y1="88.5" x2="30.12" y2="92.54" width="0" layer="19" extent="1-1"/>
-<wire x1="6.55" y1="77.785" x2="7.95" y2="82" width="0" layer="19" extent="1-1"/>
-<wire x1="6.215" y1="77.225" x2="6.55" y2="77.785" width="0" layer="19" extent="1-1"/>
+<wire x1="6.55" y1="77.785" x2="6.215" y2="77.225" width="0" layer="19" extent="1-1"/>
 <wire x1="15.51" y1="54.07" x2="10.5" y2="77.95" width="0" layer="19" extent="1-1"/>
 <wire x1="23.5" y1="56.765" x2="15.51" y2="54.07" width="0" layer="19" extent="1-1"/>
@@
 <contactref element="U2" pad="2"/>
 <via x="4.8" y="80.8" extent="1-16" drill="0.35"/>
-<wire x1="4.8" y1="80.8" x2="8.2" y2="80.8" width="0.3" layer="16"/>
-<wire x1="10.8" y1="78.2" x2="8.2" y2="80.8" width="0.3" layer="16"/>
+<wire x1="4.8" y1="80.8" x2="9" y2="80.8" width="0.3" layer="16"/>
+<wire x1="10.8" y1="79" x2="9" y2="80.8" width="0.3" layer="16"/>
 <via x="10.8" y="74.1" extent="1-16" drill="0.35"/>
-<wire x1="10.8" y1="74.1" x2="10.8" y2="78.2" width="0.3" layer="16"/>
+<wire x1="10.8" y1="74.1" x2="10.8" y2="79" width="0.3" layer="16"/>
 <wire x1="10.8" y1="74.1" x2="10.8" y2="65.3" width="0.3" layer="1"/>
 <wire x1="10.8" y1="65.3" x2="13.4" y2="62.7" width="0.3" layer="16"/>
@@
 <wire x1="6" y1="74.1" x2="10.8" y2="74.1" width="0.2" layer="1"/>
 <wire x1="4.8" y1="80.8" x2="4.8" y2="82.644975" width="0.3" layer="1"/>
-<wire x1="4.8" y1="82.644975" x2="5.0775125" y2="82.9224875" width="0.3" layer="1"/>
-<wire x1="5.0775125" y1="82.9224875" x2="5.255025" y2="83.1" width="0.3" layer="1"/>
-<wire x1="5.255025" y1="83.1" x2="5.355025" y2="83.2" width="0.3" layer="1"/>
+<wire x1="4.8" y1="82.644975" x2="5.355025" y2="83.2" width="0.3" layer="1"/>
 <wire x1="5.355025" y1="83.2" x2="5.9" y2="83.2" width="0.3" layer="1"/>
 </signal>
@@
 <wire x1="13.16" y1="67.14" x2="11.9" y2="68.4" width="0.3" layer="1"/>
 <wire x1="11.9" y1="68.4" x2="11.9" y2="75" width="0.3" layer="1"/>
-<wire x1="11.9" y1="75" x2="11.9" y2="78.9" width="0.3" layer="1"/>
-<wire x1="11.9" y1="78.9" x2="11" y2="79.8" width="0.3" layer="1"/>
-<wire x1="11" y1="79.8" x2="3.6" y2="79.8" width="0.3" layer="1"/>
+<wire x1="11.9" y1="75" x2="11.9" y2="78.5" width="0.3" layer="1"/>
+<wire x1="11.9" y1="78.5" x2="11.2" y2="79.2" width="0.3" layer="1"/>
+<wire x1="11.2" y1="79.2" x2="4.2" y2="79.2" width="0.3" layer="1"/>
 <contactref element="U2" pad="3"/>
 <via x="22.5" y="59.1" extent="1-16" drill="0.35"/>
@@
 <wire x1="4" y1="84.1" x2="2.8" y2="82.9" width="0.3" layer="1"/>
 <wire x1="2.8" y1="82.9" x2="2.8" y2="80.6" width="0.3" layer="1"/>
-<wire x1="2.8" y1="80.6" x2="3.6" y2="79.8" width="0.3" layer="1"/>
+<wire x1="2.8" y1="80.6" x2="4.2" y2="79.2" width="0.3" layer="1"/>
 <wire x1="7" y1="76.215" x2="7" y2="75.3" width="0.2" layer="1"/>
 <wire x1="7" y1="75.3" x2="7.4" y2="74.9" width="0.2" layer="1"/>
@@
 <wire x1="11.6" y1="24.3" x2="1.8" y2="24.3" width="0.2" layer="15"/>
 <wire x1="1.8" y1="24.3" x2="1" y2="25.1" width="0.2" layer="15"/>
-<wire x1="1" y1="25.1" x2="1" y2="78" width="0.2" layer="15"/>
-<wire x1="1" y1="78" x2="2" y2="79" width="0.2" layer="15"/>
-<wire x1="13.18" y1="79" x2="14.88" y2="77.3" width="0.2" layer="15"/>
-<wire x1="2" y1="79" x2="13.18" y2="79" width="0.2" layer="15"/>
+<wire x1="1" y1="25.1" x2="1" y2="71.9" width="0.2" layer="15"/>
+<wire x1="14.88" y1="77.3" x2="13.5322" y2="75.9522" width="0.2" layer="15"/>
+<wire x1="13.5322" y1="75.9522" x2="13.5322" y2="74.7967125" width="0.2" layer="15"/>
+<wire x1="13.5322" y1="74.7967125" x2="12.0254875" y2="73.29" width="0.2" layer="15"/>
+<wire x1="12.0254875" y1="73.29" x2="3" y2="73.29" width="0.2" layer="15"/>
+<wire x1="3" y1="73.29" x2="2.879875" y2="73.29" width="0.2" layer="15"/>
+<wire x1="2.879875" y1="73.29" x2="2.39" y2="73.29" width="0.2" layer="15"/>
+<wire x1="2.39" y1="73.29" x2="1" y2="71.9" width="0.2" layer="15"/>
 </signal>
 <signal name="VTX_TX">
@@
 <wire x1="12.9" y1="25" x2="2.3" y2="25" width="0.2" layer="15"/>
 <wire x1="2.3" y1="25" x2="1.6" y2="25.7" width="0.2" layer="15"/>
-<wire x1="1.6" y1="25.7" x2="1.6" y2="72.3" width="0.2" layer="15"/>
-<wire x1="1.6" y1="72.3" x2="2.3" y2="73" width="0.2" layer="15"/>
-<wire x1="13.12" y1="73" x2="14.88" y2="74.76" width="0.2" layer="15"/>
-<wire x1="2.3" y1="73" x2="13.12" y2="73" width="0.2" layer="15"/>
+<wire x1="1.6" y1="25.7" x2="1.6" y2="71.6" width="0.2" layer="15"/>
+<wire x1="1.6" y1="71.6" x2="2.7" y2="72.7" width="0.2" layer="15"/>
+<wire x1="12.82" y1="72.7" x2="14.88" y2="74.76" width="0.2" layer="15"/>
+<wire x1="2.7" y1="72.7" x2="12.82" y2="72.7" width="0.2" layer="15"/>
 </signal>
 <signal name="TELEM_RX">
@@
 <wire x1="4" y1="26.6" x2="3" y2="27.6" width="0.2" layer="15"/>
 <wire x1="3" y1="27.6" x2="3" y2="70" width="0.2" layer="15"/>
-<wire x1="3" y1="70" x2="4.3" y2="71.3" width="0.2" layer="15"/>
-<wire x1="13.26" y1="71.3" x2="14.88" y2="69.68" width="0.2" layer="15"/>
-<wire x1="4.3" y1="71.3" x2="13.26" y2="71.3" width="0.2" layer="15"/>
+<wire x1="3" y1="70" x2="4.6" y2="71.6" width="0.2" layer="15"/>
+<wire x1="12.96" y1="71.6" x2="14.88" y2="69.68" width="0.2" layer="15"/>
+<wire x1="4.6" y1="71.6" x2="12.96" y2="71.6" width="0.2" layer="15"/>
 </signal>
 <signal name="N$9">
