File: PCB/CertStack/CertStack.brd (EAGLE design)
At the start: 45 x 100 mm, 39 parts, among them J1 MEM2075-00-140-01-A, Q1 SI2302, Q2 SI2302, Q3 SI2302, Q4 SI2302, Q5 MMBT2222A, T1 DMP3098L-7, U2 INVENSENSE_ICM-20608-GINVENSE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, U3 SST26VF064B-104V/MN, U4 LT1374CS8-5PBF

Commit message: PCB
Parts:
- removed BATTERY: (no value), pinhead:1X02
- added U$2: PWR-AWG18, mylibrary:PWR-AWG18
- moved U4 10.8 mm to (41.9, 52.6)
Connections:
- new net CS_ACCEL: U$1.15
- new net CS_SD: U$1.14
- net CS-SD: no longer U$1.14
- net GND: now also U$2.-; no longer BATTERY.2
- net VCC: now also U$2.+; no longer BATTERY.1
Routing:
- net +3V3: track 68.0 -> 106.8 mm, vias 4 -> 5
- net CS_ACCEL: track 0.00 -> 22.5 mm
Changed lines of the file:
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@@
 <attribute name="PURCHASE-URL" value="https://pricing.snapeda.com/search/part/SST26VF064B-104V/MN/?ref=eda" x="-33.64" y="14.34" size="1.778" layer="27" rot="R270" display="off"/>
 </element>
-<element name="U4" library="LT1374CS8-5PBF" package="SO-8_S" value="LT1374CS8-5PBF" x="51.88" y="48.63" smashed="yes">
-<attribute name="AVAILABILITY" value="In Stock" x="123" y="-39" size="1.778" layer="27" display="off"/>
-<attribute name="DESCRIPTION" value=" Buck, SEPIC Switching Regulator IC Positive Fixed 5V 1 Output 4.5A (Switch) 8-SOIC (0.154, 3.90mm Width) " x="123" y="-39" size="1.778" layer="27" display="off"/>
-<attribute name="MF" value="Analog Devices" x="123" y="-39" size="1.778" layer="27" display="off"/>
-<attribute name="MP" value="LT1374CS8-5#PBF" x="123" y="-39" size="1.778" layer="27" display="off"/>
-<attribute name="NAME" x="48.4256" y="51.5017" size="0.4" layer="25"/>
-<attribute name="PACKAGE" value="SOIC -8 Analog Devices" x="123" y="-39" size="1.778" layer="27" display="off"/>
-<attribute name="PRICE" value="None" x="123" y="-39" size="1.778" layer="27" display="off"/>
-<attribute name="PURCHASE-URL" value="https://pricing.snapeda.com/search/part/LT1374CS8-5#PBF/?ref=eda" x="123" y="-39" size="1.778" layer="27" display="off"/>
-<attribute name="VALUE" x="48.4256" y="45.7583" size="0.4" layer="27" align="top-left"/>
+<element name="U4" library="LT1374CS8-5PBF" package="SO-8_S" value="LT1374CS8-5PBF" x="41.88" y="52.63" smashed="yes">
+<attribute name="AVAILABILITY" value="In Stock" x="113" y="-35" size="1.778" layer="27" display="off"/>
+<attribute name="DESCRIPTION" value=" Buck, SEPIC Switching Regulator IC Positive Fixed 5V 1 Output 4.5A (Switch) 8-SOIC (0.154, 3.90mm Width) " x="113" y="-35" size="1.778" layer="27" display="off"/>
+<attribute name="MF" value="Analog Devices" x="113" y="-35" size="1.778" layer="27" display="off"/>
+<attribute name="MP" value="LT1374CS8-5#PBF" x="113" y="-35" size="1.778" layer="27" display="off"/>
+<attribute name="NAME" x="38.4256" y="55.5017" size="0.4" layer="25"/>
+<attribute name="PACKAGE" value="SOIC -8 Analog Devices" x="113" y="-35" size="1.778" layer="27" display="off"/>
+<attribute name="PRICE" value="None" x="113" y="-35" size="1.778" layer="27" display="off"/>
+<attribute name="PURCHASE-URL" value="https://pricing.snapeda.com/search/part/LT1374CS8-5#PBF/?ref=eda" x="113" y="-35" size="1.778" layer="27" display="off"/>
+<attribute name="VALUE" x="38.4256" y="49.7583" size="0.4" layer="27" align="top-left"/>
 </element>
 <element name="LS1" library="mylibrary" package="CMT-8540S" value="CMT-8540S" x="38" y="69" smashed="yes"/>
@@
 <attribute name="POPULARITY" value="85" x="37" y="61" size="1.778" layer="27" rot="R180" display="off"/>
 <attribute name="SPICEPREFIX" value="R" x="37" y="61" size="1.778" layer="27" rot="R180" display="off"/>
-</element>
-<element name="BATTERY" library="pinhead" library_urn="urn:adsk.eagle:library:325" package="1X02" package3d_urn="urn:adsk.eagle:package:22435/2" value="" x="39" y="36" smashed="yes">
-<attribute name="NAME" x="36.3838" y="37.8288" size="1.27" layer="25" ratio="10"/>
-<attribute name="POPULARITY" value="98" x="39" y="36" size="1.778" layer="27" display="off"/>
-<attribute name="VALUE" x="36.46" y="32.825" size="1.27" layer="27"/>
 </element>
 <element name="Q1" library="SI2302" package="SOT23" value="SI2302" x="5" y="37" smashed="yes" rot="R180">
@@
 <attribute name="NAME" x="32.5" y="33.445" size="1.27" layer="21" align="bottom-center"/>
 </element>
+<element name="U$2" library="mylibrary" package="PWR-AWG18" value="PWR-AWG18" x="1" y="-3" smashed="yes"/>
 </elements>
 <signals>
@@
 <contactref element="LED2" pad="C"/>
 <contactref element="LED3" pad="C"/>
-<contactref element="BATTERY" pad="2"/>
 <contactref element="C2" pad="2"/>
 <contactref element="BMP384_1" pad="3"/>
@@
 <contactref element="VTX" pad="6"/>
 <contactref element="TELEM" pad="6"/>
+<contactref element="U$2" pad="-"/>
 <wire x1="41.05" y1="86" x2="41.05" y2="90" width="0" layer="19" extent="1-1"/>
 <wire x1="41.05" y1="82" x2="41.05" y2="86" width="0" layer="19" extent="1-1"/>
@@
 <wire x1="22.5" y1="64.6" x2="28.82" y2="59.49" width="0" layer="19" extent="1-1"/>
 <wire x1="4.51" y1="60.95" x2="13.51" y2="60.95" width="0" layer="19" extent="1-1"/>
+<wire x1="39.4162" y1="50.725" x2="29.62" y2="54.84" width="0" layer="19" extent="1-1"/>
 <wire x1="13.51" y1="44.8" x2="21.74" y2="51.63" width="0" layer="19" extent="1-1"/>
 <wire x1="14.05" y1="41" x2="13.51" y2="44.8" width="0" layer="19" extent="1-1"/>
@@
 <wire x1="27.5" y1="9" x2="27.5" y2="19" width="0" layer="19" extent="1-1"/>
 <wire x1="17.5" y1="19" x2="17.5" y2="29" width="0" layer="19" extent="1-1"/>
-<wire x1="49.4162" y1="46.725" x2="29.62" y2="54.84" width="0" layer="19" extent="1-1"/>
-<wire x1="40.27" y1="36" x2="49.4162" y2="46.725" width="0" layer="19" extent="1-1"/>
 <wire x1="3.5" y1="76.05" x2="4.51" y2="60.95" width="0" layer="19" extent="1-1"/>
 <wire x1="6.55" y1="76.215" x2="3.5" y2="76.05" width="0" layer="19" extent="1-1"/>
@@
 <wire x1="5.095" y1="91.9" x2="6.05" y2="82" width="0" layer="19" extent="1-1"/>
 <wire x1="14.88" y1="97.62" x2="5.095" y2="91.9" width="0" layer="19" extent="1-1"/>
+<wire x1="2.75" y1="-3" x2="17.5" y2="19" width="0" layer="19" extent="1-1"/>
 </signal>
 <signal name="+3V3">
@@
 <wire x1="6.4" y1="90.3" x2="6.4" y2="93.2" width="0.3" layer="16"/>
 <wire x1="6.215" y1="77.225" x2="5.54" y2="77.9" width="0.2" layer="1"/>
+<wire x1="5.54" y1="77.9" x2="5.52" y2="77.92" width="0.2" layer="1"/>
 <wire x1="10.5" y1="77.95" x2="9.95" y2="78.5" width="0.2" layer="1"/>
-<wire x1="9.95" y1="78.5" x2="6.8" y2="78.5" width="0.2" layer="1"/>
-<wire x1="6.8" y1="78.5" x2="6.55" y2="78.25" width="0.2" layer="1"/>
-<wire x1="6.55" y1="78.25" x2="6.55" y2="77.785" width="0.2" layer="1"/>
+<wire x1="9.95" y1="78.5" x2="6.5" y2="78.5" width="0.2" layer="1"/>
 <via x="8.2" y="80" extent="1-16" drill="0.35"/>
+<wire x1="6.5" y1="78.5" x2="6.1" y2="78.5" width="0.2" layer="1"/>
 <wire x1="8.2" y1="80" x2="8.2" y2="81.75" width="0.3" layer="1"/>
 <wire x1="8.2" y1="81.75" x2="7.95" y2="82" width="0.3" layer="1"/>
@@
 <wire x1="4.9" y1="77.9" x2="7" y2="80" width="0.2" layer="16"/>
 <wire x1="7" y1="80" x2="8.2" y2="80" width="0.2" layer="16"/>
+<wire x1="4.9" y1="63.8" x2="4.9" y2="77.9" width="0.2" layer="16"/>
+<wire x1="5.52" y1="77.92" x2="6.1" y2="78.5" width="0.2" layer="1"/>
+<wire x1="6.55" y1="77.785" x2="6.55" y2="78.45" width="0.2" layer="1"/>
+<wire x1="6.55" y1="78.45" x2="6.5" y2="78.5" width="0.2" layer="1"/>
+<via x="18" y="54.1" extent="1-16" drill="0.35"/>
+<wire x1="18" y1="54.1" x2="17.97" y2="54.07" width="0.3" layer="1"/>
+<wire x1="17.97" y1="54.07" x2="15.51" y2="54.07" width="0.3" layer="1"/>
+<wire x1="18" y1="54.1" x2="8.4" y2="54.1" width="0.2" layer="16"/>
+<wire x1="7.4" y1="61.3" x2="4.9" y2="63.8" width="0.2" layer="16"/>
+<wire x1="8.4" y1="54.1" x2="7.4" y2="55.1" width="0.2" layer="16"/>
+<wire x1="7.4" y1="55.1" x2="7.4" y2="61.3" width="0.2" layer="16"/>
 <wire x1="11" y1="88.5" x2="30.12" y2="92.54" width="0" layer="19" extent="1-1"/>
-<wire x1="6.55" y1="77.785" x2="6.215" y2="77.225" width="0" layer="19" extent="1-1"/>
-<wire x1="15.51" y1="54.07" x2="10.5" y2="77.95" width="0" layer="19" extent="1-1"/>
-<wire x1="23.5" y1="56.765" x2="15.51" y2="54.07" width="0" layer="19" extent="1-1"/>
-<wire x1="29.5" y1="29" x2="23.765" y2="56" width="0" layer="19" extent="1-1"/>
+<wire x1="23.765" y1="56" x2="18" y2="54.1" width="0" layer="19" extent="1-1"/>
+<wire x1="29.5" y1="29" x2="18" y2="54.1" width="0" layer="19" extent="1-1"/>
 </signal>
 <signal name="CS_BAR">
@@
 <signal name="CS-SD">
 <contactref element="J1" pad="P2"/>
-<contactref element="U$1" pad="14"/>
-<wire x1="30.12" y1="67.14" x2="15.51" y2="51.87" width="0" layer="19" extent="1-1"/>
-</signal>
-<signal name="VCC">
-<contactref element="BATTERY" pad="1"/>
 </signal>
 <signal name="N$19">
@@
 <wire x1="6.4322" y1="81.5322" x2="6.5" y2="81.6" width="0.2" layer="16"/>
 <wire x1="4.4967125" y1="81.5322" x2="6.4322" y2="81.5322" width="0.2" layer="16"/>
-<wire x1="4.0678" y1="63.6322" x2="4.0678" y2="81.1032875" width="0.2" layer="16"/>
+<wire x1="4.0678" y1="63.1322" x2="4.0678" y2="81.1032875" width="0.2" layer="16"/>
 <wire x1="6.5" y1="81.6" x2="13.12" y2="81.6" width="0.2" layer="16"/>
 <wire x1="13.12" y1="81.6" x2="14.88" y2="79.84" width="0.2" layer="16"/>
-<wire x1="6.7" y1="46" x2="6.7" y2="61" width="0.2" layer="16"/>
-<wire x1="6.7" y1="61" x2="4.0678" y2="63.6322" width="0.2" layer="16"/>
+<wire x1="6.7" y1="46" x2="6.7" y2="60.5" width="0.2" layer="16"/>
+<wire x1="6.7" y1="60.5" x2="4.0678" y2="63.1322" width="0.2" layer="16"/>
 </signal>
 <signal name="FET4">
@@
 <contactref element="POWER" pad="5"/>
 </signal>
+<signal name="CS_ACCEL">
+<contactref element="U$1" pad="15"/>
+<wire x1="12.8875" y1="65.8875" x2="11" y2="64" width="0.2" layer="1"/>
+<wire x1="16.19880625" y1="65.8875" x2="12.8875" y2="65.8875" width="0.2" layer="1"/>
+<wire x1="30.12" y1="69.68" x2="19.99130625" y2="69.68" width="0.2" layer="1"/>
+<wire x1="19.99130625" y1="69.68" x2="16.19880625" y2="65.8875" width="0.2" layer="1"/>
+<wire x1="11" y1="64" x2="10" y2="64" width="0.2" layer="1"/>
+</signal>
+<signal name="CS_SD">
+<contactref element="U$1" pad="14"/>
+</signal>
+<signal name="VCC">
+<contactref element="U$2" pad="+"/>
+</signal>
 </signals>
