File: PCB/CertStack/CertStack.brd (EAGLE design)
At the start: 45 x 100 mm, 39 parts, among them J1 MEM2075-00-140-01-A, Q1 SI2302, Q2 SI2302, Q3 SI2302, Q4 SI2302, Q5 MMBT2222A, T1 DMP3098L-7, U2 INVENSENSE_ICM-20608-GINVENSE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, U3 SST26VF064B-104V/MN, U4 LT1374CS8-5PBF

Commit message: PCB
Parts:
- removed U4: LT1374CS8-5PBF, LT1374CS8-5PBF:SO-8_S
- added C10, C11: 10uF, SparkFun-Capacitors:1206
- added C4: (no value), rcl:C0805
- added CC: 1.5nF, rcl:C0805
- added D1: 1N4004, diode:DO41-10
- added D2: 30V 100mA, diode:DO35Z10
- added U1: LT1374CS8-5PBF, LT1374CS8-5PBF:SO-8_S
- moved U$2 54.6 mm to (37.0, 38.0)
Connections:
- removed net SW+: POWER.5
- removed net SW-: POWER.6
- removed net V_BAT: U4.1
- new net BOOST: C4.2, D2.A, U1.2
- new net OUT: D2.C
- new net SENSE: D1.C, U1.3, U1.5
- new net SHDN: POWER.6, U1.7
- new net VC: CC.1, U1.6
- new net VSW: C4.1, U1.8
- net BATV: now also C10.1, C11.1, U1.1
- net GND: now also C10.2, C11.2, CC.2, D1.A, POWER.5, U1.4; no longer U4.4

Commit message: PCB
Parts:
- removed D2: 30V 100mA, diode:DO35Z10
- added U$3: DO-214AB, DO-214AB:DO-214AB
Connections:
- removed net OUT: D2.C
- net BOOST: no longer D2.A
Changed lines of the file:
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@@
 <attribute name="VALUE" x="36.5456" y="48.1283" size="0.4" layer="27" align="top-left"/>
-</element>
-<element name="D2" library="diode" library_urn="urn:adsk.eagle:library:210" package="DO35Z10" package3d_urn="urn:adsk.eagle:package:43342/1" value="30V 100mA" x="54" y="45" smashed="yes">
-<attribute name="NAME" x="51.714" y="46.27" size="1.27" layer="25" ratio="10"/>
-<attribute name="POPULARITY" value="1" x="54" y="45" size="1.778" layer="27" display="off"/>
-<attribute name="VALUE" x="51.714" y="42.46" size="1.27" layer="27" ratio="10"/>
 </element>
 <element name="C4" library="rcl" library_urn="urn:adsk.eagle:library:334" package="C0805" package3d_urn="urn:adsk.eagle:package:23617/2" value="" x="49" y="30" smashed="yes">
@@
 <attribute name="PROD_ID" value="CAP-10057" x="37" y="41" size="1.778" layer="27" display="off"/>
 <attribute name="VALUE" x="37" y="39.857" size="0.6096" layer="27" font="vector" ratio="20" align="top-center"/>
+</element>
+<element name="U$3" library="DO-214AB" package="DO-214AB" value="DO-214AB" x="5" y="-4" smashed="yes">
+<attribute name="AVAILABILITY" value="Not in stock" x="5" y="-4" size="1.778" layer="27" display="off"/>
+<attribute name="DESCRIPTION" value=" 143.85V Clamp 11.1A Ipp Tvs Diode Surface Mount DO-214AB (SMCJ) " x="5" y="-4" size="1.778" layer="27" display="off"/>
+<attribute name="MF" value="Littelfuse Inc." x="5" y="-4" size="1.778" layer="27" display="off"/>
+<attribute name="MP" value="DO-214AB" x="5" y="-4" size="1.778" layer="27" display="off"/>
+<attribute name="NAME" x="-0.842" y="-3.3" size="0.4" layer="25"/>
+<attribute name="PACKAGE" value="DO-214AB-214 Littelfuse Inc." x="5" y="-4" size="1.778" layer="27" display="off"/>
+<attribute name="PRICE" value="None" x="5" y="-4" size="1.778" layer="27" display="off"/>
+<attribute name="VALUE" x="-0.842" y="-4.7" size="0.4" layer="27" align="top-left"/>
 </element>
 </elements>
@@
 <signal name="BOOST">
 <contactref element="U1" pad="2"/>
-<contactref element="D2" pad="A"/>
 <contactref element="C4" pad="2"/>
-<wire x1="59.08" y1="45" x2="49.95" y2="30" width="0" layer="19" extent="1-1"/>
-<wire x1="37.5362" y1="51.635" x2="59.08" y2="45" width="0" layer="19" extent="1-1"/>
-</signal>
-<signal name="OUT">
-<contactref element="D2" pad="C"/>
+<wire x1="49.95" y1="30" x2="37.5362" y2="51.635" width="0" layer="19" extent="1-1"/>
 </signal>
 <signal name="VSW">

Commit message: PCB
Parts:
- removed U$3: DO-214AB, DO-214AB:DO-214AB
- added C3: (no value), rcl:C0805
- added D2: DO-214AB, DO-214AB:DO-214AB
- D1: value 1N4004 -> PMEG4020ETP,115; device diode:DO41-10 -> PMEG4020ETP_115:SODFL4725X110N
- moved D1 24.3 mm to (30.0, 50.0)
Connections:
- removed net SENSE: D1.C, U1.3, U1.5
- new net OUT: C3.1, D2.IN, U1.3, U1.5
- net BOOST: now also D2.OUT
- net GND: now also C3.2, D1.2; no longer D1.A
- net VSW: now also D1.1
Changed lines of the file:
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@@
 <attribute name="VALUE" x="60.73" y="34.46" size="1.27" layer="27"/>
-</element>
-<element name="D1" library="diode" library_urn="urn:adsk.eagle:library:210" package="DO41-10" package3d_urn="urn:adsk.eagle:package:43336/1" value="1N4004" x="54" y="54" smashed="yes">
-<attribute name="NAME" x="51.968" y="55.651" size="1.27" layer="25" ratio="10"/>
-<attribute name="POPULARITY" value="82" x="54" y="28" size="1.778" layer="27" display="off"/>
-<attribute name="VALUE" x="51.968" y="51.206" size="1.27" layer="27" ratio="10"/>
 </element>
 <element name="C10" library="SparkFun-Capacitors" library_urn="urn:adsk.eagle:library:510" package="1206" package3d_urn="urn:adsk.eagle:package:37426/1" value="10uF" x="37" y="45" smashed="yes">
@@
 <attribute name="VALUE" x="37" y="39.857" size="0.6096" layer="27" font="vector" ratio="20" align="top-center"/>
 </element>
-<element name="U$3" library="DO-214AB" package="DO-214AB" value="DO-214AB" x="5" y="-4" smashed="yes">
-<attribute name="AVAILABILITY" value="Not in stock" x="5" y="-4" size="1.778" layer="27" display="off"/>
-<attribute name="DESCRIPTION" value=" 143.85V Clamp 11.1A Ipp Tvs Diode Surface Mount DO-214AB (SMCJ) " x="5" y="-4" size="1.778" layer="27" display="off"/>
-<attribute name="MF" value="Littelfuse Inc." x="5" y="-4" size="1.778" layer="27" display="off"/>
-<attribute name="MP" value="DO-214AB" x="5" y="-4" size="1.778" layer="27" display="off"/>
-<attribute name="NAME" x="-0.842" y="-3.3" size="0.4" layer="25"/>
-<attribute name="PACKAGE" value="DO-214AB-214 Littelfuse Inc." x="5" y="-4" size="1.778" layer="27" display="off"/>
-<attribute name="PRICE" value="None" x="5" y="-4" size="1.778" layer="27" display="off"/>
-<attribute name="VALUE" x="-0.842" y="-4.7" size="0.4" layer="27" align="top-left"/>
+<element name="D2" library="DO-214AB" package="DO-214AB" value="DO-214AB" x="29" y="44" smashed="yes">
+<attribute name="AVAILABILITY" value="Not in stock" x="29" y="44" size="1.778" layer="27" display="off"/>
+<attribute name="DESCRIPTION" value=" 143.85V Clamp 11.1A Ipp Tvs Diode Surface Mount DO-214AB (SMCJ) " x="29" y="44" size="1.778" layer="27" display="off"/>
+<attribute name="MF" value="Littelfuse Inc." x="29" y="44" size="1.778" layer="27" display="off"/>
+<attribute name="MP" value="DO-214AB" x="29" y="44" size="1.778" layer="27" display="off"/>
+<attribute name="NAME" x="23.158" y="44.7" size="0.4" layer="25"/>
+<attribute name="PACKAGE" value="DO-214AB-214 Littelfuse Inc." x="29" y="44" size="1.778" layer="27" display="off"/>
+<attribute name="PRICE" value="None" x="29" y="44" size="1.778" layer="27" display="off"/>
+<attribute name="VALUE" x="23.158" y="43.3" size="0.4" layer="27" align="top-left"/>
+</element>
+<element name="D1" library="PMEG4020ETP_115" package="SODFL4725X110N" value="PMEG4020ETP,115" x="30" y="50" smashed="yes">
+<attribute name="AVAILABILITY" value="In Stock" x="30" y="50" size="1.778" layer="27" display="off"/>
+<attribute name="DESCRIPTION" value=" Diode Schottky 40 V 2A Surface Mount SOD-128/CFP5 " x="30" y="50" size="1.778" layer="27" display="off"/>
+<attribute name="MF" value="Nexperia USA Inc." x="30" y="50" size="1.778" layer="27" display="off"/>
+<attribute name="MP" value="PMEG4020ETP,115" x="30" y="50" size="1.778" layer="27" display="off"/>
+<attribute name="NAME" x="26.65" y="52.95" size="1.27" layer="25"/>
+<attribute name="PACKAGE" value="SOD-128 Nexperia USA" x="30" y="50" size="1.778" layer="27" display="off"/>
+<attribute name="PRICE" value="None" x="30" y="50" size="1.778" layer="27" display="off"/>
+<attribute name="PURCHASE-URL" value="https://pricing.snapeda.com/search/part/PMEG4020ETP,115/?ref=eda" x="30" y="50" size="1.778" layer="27" display="off"/>
+<attribute name="VALUE" x="26.65" y="47.05" size="1.27" layer="27" align="top-left"/>
+</element>
+<element name="C3" library="rcl" library_urn="urn:adsk.eagle:library:334" package="C0805" package3d_urn="urn:adsk.eagle:package:23617/2" value="" x="1" y="-4" smashed="yes">
+<attribute name="NAME" x="-0.27" y="-2.73" size="1.27" layer="25"/>
+<attribute name="POPULARITY" value="63" x="1" y="-4" size="1.778" layer="27" display="off"/>
+<attribute name="SPICEPREFIX" value="C" x="1" y="-4" size="1.778" layer="27" display="off"/>
+<attribute name="VALUE" x="-0.27" y="-6.54" size="1.27" layer="27"/>
 </element>
 </elements>
@@
 <contactref element="U$2" pad="-"/>
 <contactref element="U1" pad="4"/>
-<contactref element="CC" pad="2"/>
-<contactref element="D1" pad="A"/>
 <contactref element="C11" pad="2"/>
 <contactref element="C10" pad="2"/>
 <contactref element="POWER" pad="5"/>
+<contactref element="CC" pad="2"/>
+<contactref element="C3" pad="2"/>
+<contactref element="D1" pad="2"/>
 <wire x1="41.05" y1="86" x2="41.05" y2="90" width="0" layer="19" extent="1-1"/>
 <wire x1="41.05" y1="82" x2="41.05" y2="86" width="0" layer="19" extent="1-1"/>
@@
 <wire x1="23.765" y1="55.5" x2="26.52" y2="54.84" width="0" layer="19" extent="1-1"/>
 <wire x1="21.74" y1="51.63" x2="22" y2="54.235" width="0" layer="19" extent="1-1"/>
+<wire x1="32.2" y1="50" x2="29.62" y2="54.84" width="0" layer="19" extent="1-1"/>
+<wire x1="37.5362" y1="49.095" x2="32.2" y2="50" width="0" layer="19" extent="1-1"/>
+<wire x1="38.4" y1="45" x2="37.5362" y2="49.095" width="0" layer="19" extent="1-1"/>
+<wire x1="38.4" y1="41" x2="38.4" y2="45" width="0" layer="19" extent="1-1"/>
+<wire x1="38.75" y1="38" x2="38.4" y2="41" width="0" layer="19" extent="1-1"/>
 <wire x1="15.51" y1="56.27" x2="21.235" y2="55.5" width="0" layer="19" extent="1-1"/>
 <wire x1="13.51" y1="60.95" x2="15.51" y2="56.27" width="0" layer="19" extent="1-1"/>
 <wire x1="22.5" y1="64.6" x2="28.82" y2="59.49" width="0" layer="19" extent="1-1"/>
 <wire x1="4.51" y1="60.95" x2="13.51" y2="60.95" width="0" layer="19" extent="1-1"/>
-<wire x1="37.5362" y1="49.095" x2="29.62" y2="54.84" width="0" layer="19" extent="1-1"/>
-<wire x1="38.4" y1="45" x2="37.5362" y2="49.095" width="0" layer="19" extent="1-1"/>
-<wire x1="38.4" y1="41" x2="38.4" y2="45" width="0" layer="19" extent="1-1"/>
-<wire x1="38.75" y1="38" x2="38.4" y2="41" width="0" layer="19" extent="1-1"/>
 <wire x1="35.5" y1="29" x2="38.75" y2="38" width="0" layer="19" extent="1-1"/>
 <wire x1="27.5" y1="29" x2="35.5" y2="29" width="0" layer="19" extent="1-1"/>
@@
 <wire x1="5.095" y1="91.9" x2="6.05" y2="82" width="0" layer="19" extent="1-1"/>
 <wire x1="14.88" y1="97.62" x2="5.095" y2="91.9" width="0" layer="19" extent="1-1"/>
-<wire x1="59.08" y1="54" x2="37.5362" y2="49.095" width="0" layer="19" extent="1-1"/>
-<wire x1="62.95" y1="37" x2="59.08" y2="54" width="0" layer="19" extent="1-1"/>
+<wire x1="62.95" y1="37" x2="38.75" y2="38" width="0" layer="19" extent="1-1"/>
+<wire x1="1.95" y1="-4" x2="17.5" y2="19" width="0" layer="19" extent="1-1"/>
 </signal>
 <signal name="+3V3">
@@
 <contactref element="U1" pad="2"/>
 <contactref element="C4" pad="2"/>
+<contactref element="D2" pad="OUT"/>
 <wire x1="49.95" y1="30" x2="37.5362" y2="51.635" width="0" layer="19" extent="1-1"/>
+<wire x1="32.302" y1="44" x2="49.95" y2="30" width="0" layer="19" extent="1-1"/>
 </signal>
 <signal name="VSW">
 <contactref element="C4" pad="1"/>
 <contactref element="U1" pad="8"/>
-<wire x1="42.4638" y1="52.905" x2="48.05" y2="30" width="0" layer="19" extent="1-1"/>
-</signal>
-<signal name="SENSE">
+<contactref element="D1" pad="1"/>
+<wire x1="27.8" y1="50" x2="42.4638" y2="52.905" width="0" layer="19" extent="1-1"/>
+<wire x1="48.05" y1="30" x2="42.4638" y2="52.905" width="0" layer="19" extent="1-1"/>
+</signal>
+<signal name="VC">
+<contactref element="U1" pad="6"/>
+<contactref element="CC" pad="1"/>
+<wire x1="42.4638" y1="50.365" x2="61.05" y2="37" width="0" layer="19" extent="1-1"/>
+</signal>
+<signal name="OUT">
+<contactref element="U1" pad="5"/>
+<contactref element="C3" pad="1"/>
+<contactref element="D2" pad="IN"/>
 <contactref element="U1" pad="3"/>
-<contactref element="U1" pad="5"/>
-<contactref element="D1" pad="C"/>
-<wire x1="37.5362" y1="50.365" x2="48.92" y2="54" width="0" layer="19" extent="1-1"/>
-<wire x1="42.4638" y1="49.095" x2="37.5362" y2="50.365" width="0" layer="19" extent="1-1"/>
-</signal>
-<signal name="VC">
-<contactref element="CC" pad="1"/>
-<contactref element="U1" pad="6"/>
-<wire x1="42.4638" y1="50.365" x2="61.05" y2="37" width="0" layer="19" extent="1-1"/>
+<wire x1="37.5362" y1="50.365" x2="42.4638" y2="49.095" width="0" layer="19" extent="1-1"/>
+<wire x1="25.698" y1="44" x2="37.5362" y2="50.365" width="0" layer="19" extent="1-1"/>
+<wire x1="0.05" y1="-4" x2="25.698" y2="44" width="0" layer="19" extent="1-1"/>
 </signal>
 </signals>

Commit message: PCB
Parts:
- removed C3: (no value), rcl:C0805
- added C12: T491X106K050AT, T491X106K050AT:CAPMP7343X430N
- moved U1 8.60 mm to (47.0, 46.0), turned to 90 degrees
- moved D2 4.00 mm to (29.0, 40.0)
- moved U$2 2.83 mm to (35.0, 36.0)
- moved D1 1.41 mm to (29.0, 49.0)
Connections:
- net GND: now also C12.2; no longer C3.2
- net OUT: now also C12.1; no longer C3.1

Commit message: PCB
Parts:
- removed R10, R11: 15, rcl:R0805
- removed U$1: TEENSY-32, mylibrary:TEENSY-32
- added R6, R9: 10k, rcl:R0805
- added U5: INVENSENSE_ICM-20608-GINVENSENSE_ICM-20608-G_0_0, InvenSense - ICM-20608-G:INVENSENSE_ICM-20608-G_0
- R1: value 10k -> 150
- R2, R3: value 10k -> 15
- R4: value 10k -> 1k
- R7: value 1k -> 10k
- R8: value 150 -> 10k
- U1: value LT1374CS8-5PBF -> TEENSY-32; device LT1374CS8-5PBF:SO-8_S -> mylibrary:TEENSY-32
- U2: value INVENSENSE_ICM-20608-GINVENSENSE_ICM-20608-G_0_0 -> LT1374CS8-5PBF; device InvenSense - ICM-20608-G:INVENSENSE_ICM-20608-G_0 -> LT1374CS8-5PBF:SO-8_S
- moved R1 57.5 mm to (35.0, 90.0), turned to 180 degrees
- moved R8 52.9 mm to (15.0, 41.0), turned to 0 degrees
- moved R2 51.5 mm to (35.0, 86.0), turned to 180 degrees
- moved U1 50.4 mm to (22.5, 90.0), turned to 0 degrees
- moved R3 45.6 mm to (35.0, 82.0), turned to 180 degrees
- moved R7 44.7 mm to (10.0, 41.0), turned to 0 degrees
- moved R4 39.9 mm to (35.0, 78.0), turned to 180 degrees
- moved U2 26.3 mm to (47.0, 46.0), turned to 90 degrees
- renumbered BMP384_1 to U4, R14 to R5, U$2 to BATT-CON
Connections:
- net +3V3: now also R1.2, U1.3V3-1, U5.1, U5.16; no longer R8.2, U$1.3V3-1, U2.1, U2.16
- net BATV: now also U2.1; no longer U1.1
- net BOOST: now also U2.2; no longer U1.2
- net BUZZER: now also R4.2, U1.17; no longer R7.2, U$1.17
- net CS_ACCEL: now also U1.15; no longer U$1.15
- net CS_FLASH: now also U1.2; no longer U$1.2
- net CS_IMU: now also U5.5; no longer U2.5
- net CS_SD: now also U1.14; no longer U$1.14
- net F1_TRIG: now also R6.2, U1.3; no longer R1.2, U$1.3
- net F2_TRIG: now also R7.2, U1.4; no longer R2.2, U$1.4
- net F3_TRIG: now also R8.2, U1.5; no longer R3.2, U$1.5
- net F4_TRIG: now also R9.2, U1.6; no longer R4.2, U$1.6
- net GND: now also R6.1, R7.1, R8.1, R9.1, U1.GND1, U1.GND3, U2.4, U5.10, U5.11, U5.12, U5.13, U5.15, U5.7, U5.8, U5.9; no longer R1.1, R2.1, R3.1, R4.1, U$1.GND1, U$1.GND3, U1.4, U2.10, U2.11, U2.12, U2.13, U2.15, U2.7, U2.8, U2.9
- net GPS_RX: now also U1.9; no longer U$1.9
- net GPS_TX: now also U1.10; no longer U$1.10
- net LED-ER: now also R3.2, U1.20; no longer R11.2, U$1.20
- net LED-HB: now also R2.2, U1.21; no longer R10.2, U$1.21
- net MISO: now also U1.12, U5.4; no longer U$1.12, U2.4
- net MOSI: now also U1.11, U5.3; no longer U$1.11, U2.3
- net N$16: now also R1.1; no longer R8.1
- net N$17: now also R2.1; no longer R10.1
- net N$22: now also R4.1; no longer R7.1
- net N$6: now also R3.1; no longer R11.1
- net N$7: now also U5.14; no longer U2.14
- net OUT: now also U2.3, U2.5; no longer U1.3, U1.5
- net SCK: now also U1.13, U5.2; no longer U$1.13, U2.2
- net SCL: now also U1.19; no longer U$1.19
- net SDA: now also U1.18; no longer U$1.18
- net SHDN: now also U2.7; no longer U1.7
- net TELEM_RX: now also U1.0; no longer U$1.0
- net TELEM_TX: now also U1.1; no longer U$1.1
- net VBUS: now also U1.VIN; no longer U$1.VIN
- net VC: now also U2.6; no longer U1.6
- net VSW: now also U2.8; no longer U1.8
- net VTX_RX: now also U1.7; no longer U$1.7
- net VTX_TX: now also U1.8; no longer U$1.8

Commit message: PCB
Parts:
- removed CC: 1.5nF, rcl:C0805
- added C3: 10uF, SparkFun-Capacitors:1206
- added U$1: IHLP3232DZER6R8M11, mylibrary:IHLP3232DZER6R8M11
- C1: value (none) -> T491X106K050AT; device rcl:C0805 -> T491X106K050AT:CAPMP7343X430N
- C10: value 10uF -> 2.2uF; device SparkFun-Capacitors:1206 -> rcl:C0805
- C11: value 10uF -> 10nF; device SparkFun-Capacitors:1206 -> rcl:C0805
- C12: value T491X106K050AT -> 0.47uF; device T491X106K050AT:CAPMP7343X430N -> rcl:C0805
- C4: value (none) -> 10uF; device rcl:C0805 -> SparkFun-Capacitors:1206
- C5: value 2.2uF -> 1.5nF
- C6: value 0.1uF -> 100nF
- C7: value 10nF -> (none)
- C8: value 0.47uF -> (none)
- C9: value 100nF -> 0.1uF
- moved C2 35.7 mm to (28.0, 51.0), turned to 0 degrees
- moved C1 34.8 mm to (39.0, 57.0), turned to 180 degrees
- moved C7 33.6 mm to (3.50, 77.0)
- moved C12 32.3 mm to (22.7, 51.6), turned to 180 degrees
- moved C6 30.7 mm to (7.00, 82.0), turned to 180 degrees
- moved C9 30.7 mm to (27.9, 59.5), turned to 0 degrees
- moved C8 28.1 mm to (10.5, 77.0), turned to 270 degrees
- moved C4 23.4 mm to (26.5, 36.4), turned to 270 degrees
- moved C11 16.5 mm to (29.6, 55.8), turned to 270 degrees
- moved C5 15.5 mm to (28.0, 40.4), turned to 0 degrees
- moved C10 15.0 mm to (26.5, 55.8), turned to 270 degrees
- moved U2 9.02 mm to (38.6, 42.7)
- moved D1 7.44 mm to (32.8, 42.6), turned to 270 degrees
- moved D2 7.21 mm to (25.0, 46.0), turned to 180 degrees
Connections:
- removed net VCC: BATT-CON.+
- net +3V3: now also C10.1, C11.1, C8.1; no longer C1.1, C2.1, C5.1
- net BATV: now also BATT-CON.+, C3.1, C4.1; no longer C10.1, C11.1
- net BOOST: now also C2.2; no longer C4.2
- net GND: now also C3.2, C4.2; no longer C2.2, CC.2
- net N$7: now also C12.1; no longer C8.1
- net OUT: now also C1.1, U$1.2; no longer C12.1
- net VC: now also C5.1; no longer CC.1
- net VSW: now also C2.1, U$1.1; no longer C4.1

Commit message: PCB. Big changes.
Parts:
- added R10, R11: ??, rcl:R0805
- moved T1 34.5 mm to (35.6, 95.1)
- moved R5 33.1 mm to (39.0, 94.0)
- moved D2 16.6 mm to (40.3, 39.5), turned to 270 degrees
- moved D1 8.80 mm to (27.6, 49.7), turned to 180 degrees
- moved C11 6.40 mm to (24.6, 59.8)
- moved C9 6.32 mm to (21.9, 61.5)
- moved U2 5.67 mm to (33.0, 41.8)
- moved C2 4.71 mm to (27.0, 46.4), turned to 180 degrees
- moved C12 4.12 mm to (18.7, 50.6)
- moved C4 2.84 mm to (27.0, 39.2), turned to 180 degrees
- moved C5 2.60 mm to (27.0, 42.8), turned to 180 degrees
- moved C3 2.53 mm to (27.0, 35.6), turned to 180 degrees
- moved BATT-CON 2.04 mm to (33.0, 35.6)
- moved C1 2.00 mm to (39.1, 59.0)
- moved U$1 1.10 mm to (39.1, 51.1)
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Connections:
- new net N$1: R10.1, R11.2
- net BATV: now also R10.2
- net GND: now also R11.1
Routing:
- net BOOST: track 0.00 -> 31.2 mm
- net OUT: track 0.00 -> 28.3 mm
- net SHDN: track 0.00 -> 22.7 mm, vias 0 -> 2
- net BATV: track 10.0 -> 26.9 mm
- net VSW: track 0.00 -> 14.6 mm
- net +5V: track 20.8 -> 7.24 mm
- net +3V3: track 106.8 -> 96.4 mm
- net VC: track 0.00 -> 7.20 mm
- net GND: track 5.90 -> 9.71 mm
- net N$12: track 3.09 -> 0.00 mm
- net VBUS: track 45.9 -> 43.9 mm
- net VIDEO: track 10.0 -> 9.00 mm
- net TELEM_TX: track 87.1 -> 88.1 mm
- net TELEM_RX: track 87.4 -> 88.4 mm
- net FET2: track 27.9 -> 26.9 mm
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
Commit message: PCB
Parts:
- moved R10 18.4 mm to (20.0, 44.5)
- moved R11 13.5 mm to (20.0, 48.0), turned to 180 degrees
- moved R5 4.00 mm to (35.0, 94.0)
- moved T1 2.88 mm to (34.0, 97.5), turned to 270 degrees
- moved C12 1.56 mm to (19.9, 51.6)
Connections:
- net +5V: now also C1.1, D2.IN, U$1.2, U2.5
- net OUT: no longer C1.1, D2.IN, U$1.2, U2.5
Routing:
- net +5V: track 7.24 -> 62.4 mm, vias 1 -> 0
- net VBUS: track 43.9 -> 2.92 mm
- net OUT: track 28.3 -> 4.47 mm
- net N$12: track 0.00 -> 2.90 mm
- net GND: vias 0 -> 1
