File: PCB/CertStack/CertStack.brd (EAGLE design)
At the start: 45 x 100 mm, 49 parts, among them J1 MEM2075-00-140-01-A, Q1 SI2302, Q2 SI2302, Q3 SI2302, Q4 SI2302, Q5 MMBT2222A, T1 DMP3098L-7, U1 TEENSY-32, U2 LT1374CS8-5PBF, U3 SST26VF064B-104V/MN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

Commit message: PCB
Connections:
- removed net OUT: U2.3
- net +5V: now also U2.3
Routing:
- net BATV: track 26.9 -> 106.6 mm, vias 0 -> 1
- net +3V3: track 96.4 -> 127.8 mm, vias 5 -> 6
- net +5V: track 62.4 -> 73.4 mm
- net OUT: track 4.47 -> 0.00 mm
Changed lines of the file:
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@@
 <contactref element="R1" pad="2"/>
 <contactref element="U1" pad="3V3-1"/>
-<wire x1="30.12" y1="92.54" x2="31.51" y2="92.54" width="0.3" layer="1"/>
-<wire x1="31.51" y1="92.54" x2="34.05" y2="90" width="0.3" layer="1"/>
 <via x="6.4" y="93.2" extent="1-16" drill="0.35"/>
 <via x="11" y="88.5" extent="1-16" drill="0.35"/>
@@
 <wire x1="8.4" y1="54.1" x2="7.4" y2="55.1" width="0.2" layer="16"/>
 <wire x1="7.4" y1="55.1" x2="7.4" y2="61.3" width="0.2" layer="16"/>
-<wire x1="11" y1="88.5" x2="30.12" y2="92.54" width="0" layer="19" extent="1-1"/>
-<wire x1="23.765" y1="56" x2="18" y2="54.1" width="0" layer="19" extent="1-1"/>
+<via x="32.3" y="90" extent="1-16" drill="0.35"/>
+<wire x1="34.05" y1="90" x2="32.3" y2="90" width="0.3" layer="1"/>
+<wire x1="32.3" y1="90" x2="32.3" y2="63.3" width="0.3" layer="16"/>
+<wire x1="18" y1="54.1" x2="25.9" y2="54.1" width="0.3" layer="16"/>
+<wire x1="32.3" y1="90" x2="30.12" y2="92.54" width="0" layer="19" extent="1-1"/>
+<wire x1="24.62" y1="60.74" x2="32.3" y2="63.3" width="0" layer="19" extent="1-16"/>
+<wire x1="20.92" y1="61.49" x2="24.62" y2="60.74" width="0" layer="19" extent="1-1"/>
+<wire x1="23.5" y1="56.765" x2="24.62" y2="60.74" width="0" layer="19" extent="1-1"/>
 <wire x1="26.52" y1="56.74" x2="23.765" y2="56" width="0" layer="19" extent="1-1"/>
-<wire x1="20.92" y1="61.49" x2="26.92" y2="57.14" width="0" layer="19" extent="1-1"/>
-<wire x1="24.62" y1="60.74" x2="26.92" y2="57.14" width="0" layer="19" extent="1-1"/>
-<wire x1="29.5" y1="28" x2="18" y2="54.1" width="0" layer="19" extent="1-1"/>
+<wire x1="25.9" y1="54.1" x2="26.52" y2="56.74" width="0" layer="19" extent="1-16"/>
+<wire x1="29.5" y1="28" x2="25.9" y2="54.1" width="0" layer="19" extent="1-16"/>
 </signal>
 <signal name="CS_BAR">
@@
 <wire x1="44" y1="68" x2="41.5" y2="65.5" width="0.4" layer="1"/>
 <wire x1="44" y1="90.3558" x2="44" y2="68" width="0.4" layer="1"/>
-<wire x1="34.905" y1="44.2638" x2="40.3" y2="42.802" width="0" layer="19" extent="1-1"/>
-<wire x1="31.5" y1="28" x2="34.905" y2="44.2638" width="0" layer="19" extent="1-1"/>
+<contactref element="U2" pad="3"/>
+<wire x1="33.635" y1="39.3362" x2="33.635" y2="41.535" width="0.5" layer="1"/>
+<wire x1="34.905" y1="42.805" x2="34.905" y2="43" width="0.5" layer="1"/>
+<wire x1="33.635" y1="41.535" x2="34.905" y2="42.805" width="0.5" layer="1"/>
+<wire x1="35.103" y1="42.802" x2="34.905" y2="43" width="0.5" layer="1"/>
+<wire x1="34.905" y1="44.2638" x2="34.905" y2="43" width="0.5" layer="1"/>
+<wire x1="40.3" y1="42.802" x2="35.103" y2="42.802" width="0.5" layer="1"/>
+<wire x1="31.5" y1="28" x2="33.635" y2="39.3362" width="0" layer="19" extent="1-1"/>
 <wire x1="9.5" y1="28" x2="31.5" y2="28" width="0" layer="19" extent="1-1"/>
 </signal>
@@
 <wire x1="33.5" y1="31.7" x2="33.5" y2="28" width="0.5" layer="1"/>
 <contactref element="R10" pad="2"/>
-<wire x1="20.95" y1="44.5" x2="34.05" y2="94" width="0" layer="19" extent="1-1"/>
+<via x="32.5" y="94" extent="1-16" drill="0.35"/>
+<wire x1="34.05" y1="94" x2="32.5" y2="94" width="0.3" layer="1"/>
+<wire x1="32.5" y1="94" x2="37" y2="94" width="0.3" layer="15"/>
+<wire x1="37" y1="94" x2="44" y2="87" width="0.3" layer="15"/>
+<wire x1="44" y1="87" x2="44" y2="38.6" width="0.3" layer="15"/>
+<wire x1="31.28829375" y1="35.6" x2="31.25" y2="35.6" width="0.3" layer="15"/>
+<wire x1="32.86329375" y1="34.025" x2="31.28829375" y2="35.6" width="0.3" layer="15"/>
+<wire x1="39.425" y1="34.025" x2="32.86329375" y2="34.025" width="0.3" layer="15"/>
+<wire x1="44" y1="38.6" x2="39.425" y2="34.025" width="0.3" layer="15"/>
 <wire x1="28.4" y1="39.2" x2="20.95" y2="44.5" width="0" layer="19" extent="1-1"/>
 <wire x1="9.5" y1="19" x2="28.4" y2="35.6" width="0" layer="19" extent="1-1"/>
@@
 <wire x1="28.25" y1="42.5" x2="27.95" y2="42.8" width="0.5" layer="1"/>
 </signal>
-<signal name="OUT">
-<contactref element="U2" pad="3"/>
-<wire x1="33.635" y1="39.3362" x2="33.635" y2="41.535" width="0.5" layer="1"/>
-<wire x1="34.905" y1="42.805" x2="34.905" y2="43" width="0.5" layer="1"/>
-<wire x1="33.635" y1="41.535" x2="34.905" y2="42.805" width="0.5" layer="1"/>
-<wire x1="35.103" y1="42.802" x2="34.905" y2="43" width="0.5" layer="1"/>
-</signal>
 <signal name="N$1">

Commit message: linear reg
Parts:
- added C13, C16, C18: 1uF, rcl:C0805
- added C14, C15: 10uF, rcl:C0805
- added U6: ADP7158ACPZ-3.3-R7, ADP7158ACPZ-3.3-R7:SON50P300X300X80-11N
Connections:
- new net N$4: C13.2, U6.4
- new net N$5: C16.1, U6.8
- new net N$8: C18.1, U6.6, U6.7
- net +3V3: now also C15.1, U6.1, U6.2, U6.3
- net +5V: now also C14.1, U6.10, U6.5, U6.9
- net GND: now also C13.1, C14.2, C15.2, C16.2, C18.2
Changed lines of the file:
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@@
 <?xml version="1.0" encoding="utf-8"?>
 <!DOCTYPE eagle SYSTEM "eagle.dtd">
-<eagle version="9.6.1">
+<eagle version="9.5.2">
 <drawing>
 <settings>
-<setting alwaysvectorfont="yes"/>
+<setting alwaysvectorfont="no"/>
 <setting verticaltext="up"/>
 </settings>
@@
 <attribute name="VALUE" x="20.635" y="50.54" size="1.27" layer="27" rot="R180"/>
 </element>
+<element name="U6" library="ADP7158ACPZ-3.3-R7" package="SON50P300X300X80-11N" value="ADP7158ACPZ-3.3-R7" x="3" y="-4" smashed="yes">
+<attribute name="AVAILABILITY" value="In Stock" x="3" y="-4" size="1.778" layer="27" display="off"/>
+<attribute name="DESCRIPTION" value=" Linear Voltage Regulator IC Positive Fixed 1 Output 2A 10-LFCSP-WD (3x3) " x="3" y="-4" size="1.778" layer="27" display="off"/>
+<attribute name="MF" value="Analog Devices" x="3" y="-4" size="1.778" layer="27" display="off"/>
+<attribute name="MP" value="ADP7158ACPZ-3.3-R7" x="3" y="-4" size="1.778" layer="27" display="off"/>
+<attribute name="NAME" x="0.66" y="-2.313" size="1.27" layer="25"/>
+<attribute name="PACKAGE" value="LFCSP -10 Analog Devices" x="3" y="-4" size="1.778" layer="27" display="off"/>
+<attribute name="PRICE" value="None" x="3" y="-4" size="1.778" layer="27" display="off"/>
+<attribute name="PURCHASE-URL" value="https://pricing.snapeda.com/search/part/ADP7158ACPZ-3.3-R7/?ref=eda" x="3" y="-4" size="1.778" layer="27" display="off"/>
+<attribute name="VALUE" x="0.66" y="-5.687" size="1.27" layer="27" align="top-left"/>
+</element>
+<element name="C13" library="rcl" library_urn="urn:adsk.eagle:library:334" package="C0805" package3d_urn="urn:adsk.eagle:package:23617/2" value="1uF" x="14" y="-11" smashed="yes">
+<attribute name="NAME" x="12.73" y="-9.73" size="1.27" layer="25"/>
+<attribute name="POPULARITY" value="63" x="2" y="-11" size="1.778" layer="27" display="off"/>
+<attribute name="SPICEPREFIX" value="C" x="2" y="-11" size="1.778" layer="27" display="off"/>
+<attribute name="VALUE" x="12.73" y="-13.54" size="1.27" layer="27"/>
+</element>
+<element name="C14" library="rcl" library_urn="urn:adsk.eagle:library:334" package="C0805" package3d_urn="urn:adsk.eagle:package:23617/2" value="10uF" x="2" y="-11" smashed="yes">
+<attribute name="NAME" x="0.73" y="-9.73" size="1.27" layer="25"/>
+<attribute name="POPULARITY" value="63" x="2" y="-18" size="1.778" layer="27" display="off"/>
+<attribute name="SPICEPREFIX" value="C" x="2" y="-18" size="1.778" layer="27" display="off"/>
+<attribute name="VALUE" x="0.73" y="-13.54" size="1.27" layer="27"/>
+</element>
+<element name="C15" library="rcl" library_urn="urn:adsk.eagle:library:334" package="C0805" package3d_urn="urn:adsk.eagle:package:23617/2" value="10uF" x="8" y="-11" smashed="yes">
+<attribute name="NAME" x="6.73" y="-9.73" size="1.27" layer="25"/>
+<attribute name="POPULARITY" value="63" x="2" y="-25" size="1.778" layer="27" display="off"/>
+<attribute name="SPICEPREFIX" value="C" x="2" y="-25" size="1.778" layer="27" display="off"/>
+<attribute name="VALUE" x="6.73" y="-13.54" size="1.27" layer="27"/>
+</element>
+<element name="C16" library="rcl" library_urn="urn:adsk.eagle:library:334" package="C0805" package3d_urn="urn:adsk.eagle:package:23617/2" value="1uF" x="2" y="-18" smashed="yes">
+<attribute name="NAME" x="0.73" y="-16.73" size="1.27" layer="25"/>
+<attribute name="POPULARITY" value="63" x="2" y="-32" size="1.778" layer="27" display="off"/>
+<attribute name="SPICEPREFIX" value="C" x="2" y="-32" size="1.778" layer="27" display="off"/>
+<attribute name="VALUE" x="0.73" y="-20.54" size="1.27" layer="27"/>
+</element>
+<element name="C18" library="rcl" library_urn="urn:adsk.eagle:library:334" package="C0805" package3d_urn="urn:adsk.eagle:package:23617/2" value="1uF" x="7" y="-18" smashed="yes">
+<attribute name="NAME" x="5.73" y="-16.73" size="1.27" layer="25"/>
+<attribute name="POPULARITY" value="63" x="2" y="-39" size="1.778" layer="27" display="off"/>
+<attribute name="SPICEPREFIX" value="C" x="2" y="-39" size="1.778" layer="27" display="off"/>
+<attribute name="VALUE" x="5.73" y="-20.54" size="1.27" layer="27"/>
+</element>
 </elements>
 <signals>
@@
 <wire x1="34.905" y1="35.755" x2="34.75" y2="35.6" width="0.5" layer="1"/>
 <contactref element="R11" pad="1"/>
+<via x="5.1" y="93.2" extent="1-16" drill="0.35"/>
+<contactref element="C15" pad="2"/>
+<contactref element="C13" pad="1"/>
+<contactref element="C16" pad="2"/>
+<contactref element="C14" pad="2"/>
+<contactref element="C18" pad="2"/>
 <wire x1="41.05" y1="86" x2="41.05" y2="90" width="0" layer="19" extent="1-1"/>
 <wire x1="41.05" y1="82" x2="41.05" y2="86" width="0" layer="19" extent="1-1"/>
@@
 <wire x1="6.05" y1="82" x2="7" y2="77.785" width="0" layer="19" extent="1-1"/>
 <wire x1="5.095" y1="91.9" x2="6.05" y2="82" width="0" layer="19" extent="1-1"/>
-<wire x1="14.88" y1="97.62" x2="5.095" y2="91.9" width="0" layer="19" extent="1-1"/>
-<via x="5.1" y="93.2" extent="1-16" drill="0.35"/>
+<wire x1="5.1" y1="93.2" x2="5.095" y2="91.9" width="0" layer="19" extent="1-1"/>
+<wire x1="14.88" y1="97.62" x2="5.1" y2="93.2" width="0" layer="19" extent="1-1"/>
+<wire x1="13.05" y1="-11" x2="27.5" y2="10" width="0" layer="19" extent="1-1"/>
+<wire x1="8.95" y1="-11" x2="13.05" y2="-11" width="0" layer="19" extent="1-1"/>
+<wire x1="2.95" y1="-11" x2="8.95" y2="-11" width="0" layer="19" extent="1-1"/>
+<wire x1="2.95" y1="-18" x2="2.95" y2="-11" width="0" layer="19" extent="1-1"/>
+<wire x1="7.95" y1="-18" x2="2.95" y2="-18" width="0" layer="19" extent="1-1"/>
 </signal>
 <signal name="+3V3">
@@
 <wire x1="32.3" y1="90" x2="32.3" y2="63.3" width="0.3" layer="16"/>
 <wire x1="18" y1="54.1" x2="25.9" y2="54.1" width="0.3" layer="16"/>
+<contactref element="U6" pad="2"/>
+<contactref element="C15" pad="1"/>
+<contactref element="U6" pad="3"/>
+<contactref element="U6" pad="1"/>
 <wire x1="32.3" y1="90" x2="30.12" y2="92.54" width="0" layer="19" extent="1-1"/>
 <wire x1="24.62" y1="60.74" x2="32.3" y2="63.3" width="0" layer="19" extent="1-16"/>
@@
 <wire x1="25.9" y1="54.1" x2="26.52" y2="56.74" width="0" layer="19" extent="1-16"/>
 <wire x1="29.5" y1="28" x2="25.9" y2="54.1" width="0" layer="19" extent="1-16"/>
+<wire x1="7.05" y1="-11" x2="29.5" y2="10" width="0" layer="19" extent="1-1"/>
+<wire x1="1.565" y1="-4" x2="7.05" y2="-11" width="0" layer="19" extent="1-1"/>
+<wire x1="1.565" y1="-3.5" x2="1.565" y2="-4" width="0" layer="19" extent="1-1"/>
+<wire x1="1.565" y1="-3" x2="1.565" y2="-3.5" width="0" layer="19" extent="1-1"/>
 </signal>
 <signal name="CS_BAR">
@@
 <wire x1="34.905" y1="44.2638" x2="34.905" y2="43" width="0.5" layer="1"/>
 <wire x1="40.3" y1="42.802" x2="35.103" y2="42.802" width="0.5" layer="1"/>
+<contactref element="U6" pad="10"/>
+<contactref element="U6" pad="9"/>
+<contactref element="C14" pad="1"/>
+<contactref element="U6" pad="5"/>
 <wire x1="31.5" y1="28" x2="33.635" y2="39.3362" width="0" layer="19" extent="1-1"/>
 <wire x1="9.5" y1="28" x2="31.5" y2="28" width="0" layer="19" extent="1-1"/>
+<wire x1="4.435" y1="-3" x2="9.5" y2="28" width="0" layer="19" extent="1-1"/>
+<wire x1="4.435" y1="-3.5" x2="4.435" y2="-3" width="0" layer="19" extent="1-1"/>
+<wire x1="1.565" y1="-5" x2="4.435" y2="-3.5" width="0" layer="19" extent="1-1"/>
+<wire x1="1.05" y1="-11" x2="1.565" y2="-5" width="0" layer="19" extent="1-1"/>
 </signal>
 <signal name="SDA">
@@
 <wire x1="19.05" y1="44.5" x2="19.05" y2="48" width="0" layer="19" extent="1-1"/>
 </signal>
+<signal name="N$4">
+<contactref element="U6" pad="4"/>
+<contactref element="C13" pad="2"/>
+<wire x1="14.95" y1="-11" x2="1.565" y2="-4.5" width="0" layer="19" extent="1-1"/>
+</signal>
+<signal name="N$5">
+<contactref element="C16" pad="1"/>
+<contactref element="U6" pad="8"/>
+<wire x1="4.435" y1="-4" x2="1.05" y2="-18" width="0" layer="19" extent="1-1"/>
+</signal>
+<signal name="N$8">
+<contactref element="U6" pad="6"/>
+<contactref element="U6" pad="7"/>
+<contactref element="C18" pad="1"/>
+<wire x1="4.435" y1="-5" x2="6.05" y2="-18" width="0" layer="19" extent="1-1"/>
+<wire x1="4.435" y1="-4.5" x2="4.435" y2="-5" width="0" layer="19" extent="1-1"/>
+</signal>
 </signals>

Commit message: PCB
Parts:
- removed C16, C18: 1uF, rcl:C0805
- added IMU1: MLX90395KDCMLX90395, MLX90395KDC:MLX90395KDC_FPRT
- C13: value 1uF -> 4.7uF
- C14: device rcl:C0805 -> SparkFun-Capacitors:1206
- C15: value 10uF -> 100nF
- U6: value ADP7158ACPZ-3.3-R7 -> ZLDO1117G33TA; device ADP7158ACPZ-3.3-R7:SON50P300X300X80-11N -> ZLDO1117G33TA:SOT230P700X180-4N
- moved C15 79.2 mm to (2.30, 68.0), turned to 90 degrees
- moved C14 66.6 mm to (28.2, 50.2), turned to 270 degrees
- moved C13 62.1 mm to (25.9, 50.0), turned to 270 degrees
- moved U6 55.8 mm to (20.6, 49.0), turned to 180 degrees
- moved R10 42.7 mm to (35.0, 84.5)
- moved R11 41.8 mm to (35.0, 87.0)
- moved C12 7.41 mm to (26.8, 54.3), turned to 0 degrees
- moved C10 4.24 mm to (27.9, 59.8), turned to 90 degrees
- moved D1 4.00 mm to (31.5, 50.6), turned to 90 degrees
- moved LED2 4.00 mm to (40.0, 82.0)
- moved R2 4.00 mm to (35.0, 82.0)
- moved LED1 3.00 mm to (40.0, 87.0)
- moved LED3 3.00 mm to (40.0, 79.0)
- moved R3 3.00 mm to (35.0, 79.0)
- moved R4 3.00 mm to (35.0, 75.0)
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Connections:
- removed net N$5: C16.1, U6.8
- removed net N$8: C18.1, U6.6, U6.7
- net +3V3: now also C13.2, IMU1.P5, IMU1.P7, IMU1.P8, U6.4; no longer U6.1, U6.3
- net +5V: now also U6.3; no longer U6.10, U6.5, U6.9
- net GND: now also IMU1.P3, IMU1.P6, U6.1; no longer C16.2, C18.2
- net N$4: now also IMU1.P4; no longer C13.2, U6.4
- net SCL: now also IMU1.P1
- net SDA: now also IMU1.P2
Routing:
- net SCL: track 0.00 -> 128.7 mm, vias 0 -> 2
- net SDA: track 0.00 -> 124.9 mm, vias 0 -> 2
- net +5V: track 73.4 -> 160.7 mm, vias 0 -> 2
- net BATV: track 106.6 -> 158.2 mm
- net +3V3: track 127.8 -> 157.5 mm
- net GND: track 9.71 -> 3.80 mm
- net N$7: track 0.00 -> 2.36 mm
- net VSW: track 14.6 -> 12.6 mm
- net N$19: track 5.81 -> 4.35 mm
- net N$16: track 3.00 -> 4.24 mm
- net LED-ER: track 4.09 -> 5.33 mm
- net BUZZER: track 5.27 -> 4.03 mm
- net LED-HB: track 4.38 -> 5.14 mm
- net MOSI: track 64.8 -> 64.1 mm

Commit message: PCB
Routing:
- net +3V3: track 157.5 -> 211.7 mm, vias 6 -> 8
- net N$1: track 0.00 -> 2.50 mm
Changed lines of the file:
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@@
 <wire x1="34.05" y1="90" x2="32.3" y2="90" width="0.3" layer="1"/>
 <wire x1="32.3" y1="90" x2="32.3" y2="63.3" width="0.3" layer="16"/>
-<wire x1="18" y1="54.1" x2="25.9" y2="54.1" width="0.3" layer="16"/>
 <contactref element="U6" pad="4"/>
 <contactref element="U6" pad="2"/>
@@
 <wire x1="2.3" y1="67.05" x2="4.345" y2="67.05" width="0.1524" layer="1"/>
 <wire x1="4.345" y1="67.05" x2="4.735" y2="66.66" width="0.1524" layer="1"/>
-<wire x1="32.3" y1="90" x2="30.12" y2="92.54" width="0" layer="19" extent="1-1"/>
-<wire x1="27.88" y1="58.86" x2="32.3" y2="63.3" width="0" layer="19" extent="1-16"/>
-<wire x1="25.9" y1="54.1" x2="23.765" y2="55.9" width="0" layer="19" extent="1-16"/>
-<wire x1="25.9" y1="49.05" x2="25.9" y2="54.1" width="0" layer="19" extent="1-16"/>
-<wire x1="17.59" y1="49" x2="18" y2="54.1" width="0" layer="19" extent="1-1"/>
-<wire x1="29.5" y1="28" x2="25.9" y2="49.05" width="0" layer="19" extent="1-1"/>
+<wire x1="27.88" y1="58.86" x2="29.34" y2="58.86" width="0.3" layer="1"/>
+<wire x1="29.34" y1="58.86" x2="29.4" y2="58.8" width="0.3" layer="1"/>
+<wire x1="29.4" y1="58.8" x2="32.35" y2="61.75" width="0.3" layer="1"/>
+<wire x1="32.35" y1="61.75" x2="32.35" y2="63.25" width="0.3" layer="1"/>
+<wire x1="32.35" y1="63.25" x2="32.3" y2="63.3" width="0.3" layer="1"/>
+<via x="32.3" y="63.3" extent="1-16" drill="0.35"/>
+<wire x1="23.61" y1="49" x2="17.59" y2="49" width="0.5" layer="1"/>
+<wire x1="17.59" y1="49" x2="18" y2="48.59" width="0.5" layer="1"/>
+<wire x1="19.1" y1="44.6" x2="20.9" y2="44.6" width="0.5" layer="1"/>
+<via x="20.9" y="44.6" extent="1-16" drill="0.35"/>
+<wire x1="20.9" y1="44.6" x2="18" y2="47.5" width="0.5" layer="16"/>
+<wire x1="18" y1="47.5" x2="18" y2="54.1" width="0.5" layer="16"/>
+<wire x1="18" y1="48.59" x2="18" y2="45.7" width="0.5" layer="1"/>
+<wire x1="18" y1="45.7" x2="19.1" y2="44.6" width="0.5" layer="1"/>
+<wire x1="32.3" y1="90" x2="32.3" y2="91.6" width="0.5" layer="16"/>
+<wire x1="32.3" y1="91.6" x2="31.36" y2="92.54" width="0.5" layer="16"/>
+<wire x1="31.36" y1="92.54" x2="30.12" y2="92.54" width="0.5" layer="16"/>
+<wire x1="8.2" y1="80" x2="13.46739375" y2="80" width="0.3" layer="2"/>
+<wire x1="13.46739375" y1="80" x2="14.41939375" y2="80.952" width="0.3" layer="2"/>
+<wire x1="18.532" y1="80.952" x2="30.12" y2="92.54" width="0.3" layer="2"/>
+<wire x1="14.41939375" y1="80.952" x2="18.532" y2="80.952" width="0.3" layer="2"/>
+<wire x1="29.5" y1="28" x2="20.9" y2="44.6" width="0" layer="19" extent="1-1"/>
 </signal>
 <signal name="CS_BAR">
@@
 <contactref element="U5" pad="14"/>
 <contactref element="C12" pad="1"/>
-<wire x1="23.765" y1="54.9" x2="25.23" y2="54.9" width="0.25" layer="1"/>
-<wire x1="25.23" y1="54.9" x2="25.86" y2="54.27" width="0.25" layer="1"/>
+<wire x1="23.765" y1="54.9" x2="25.23" y2="54.9" width="0.1524" layer="1"/>
+<wire x1="25.23" y1="54.9" x2="25.86" y2="54.27" width="0.1524" layer="1"/>
 </signal>
 <signal name="+5V">
@@
 <contactref element="R11" pad="2"/>
 <contactref element="R10" pad="1"/>
-<wire x1="34.05" y1="84.5" x2="34.05" y2="87" width="0" layer="19" extent="1-1"/>
+<wire x1="34.05" y1="84.5" x2="34.05" y2="87" width="0.3" layer="1"/>
 </signal>
 <signal name="N$4">

Commit message: PCB
Parts:
- added C16, C17: (no value), rcl:C0805
- added L1: IHLP3232DZER6R8M11, mylibrary:IHLP3232DZER6R8M11
- U$1: value IHLP3232DZER6R8M11 -> KIONIX_KXTJ3-1057; device mylibrary:IHLP3232DZER6R8M11 -> KIONIX_KXTJ3-1057:KIONIX_KXTJ3-1057
- moved U$1 63.9 mm to (-3.00, 3.00)
- moved R10 6.50 mm to (35.0, 91.0)
- moved R1 5.00 mm to (35.0, 85.0)
- moved LED1 2.00 mm to (40.0, 85.0)
- moved R11 1.00 mm to (35.0, 88.0)
- moved R4 1.00 mm to (35.0, 76.0)
Connections:
- net +3V3: now also C16.1, C17.1, U$1.3, U$1.7; no longer U1.3V3-1
- net +5V: now also L1.2; no longer U$1.2
- net GND: now also C16.2, C17.2, U$1.8, U$1.9
- net SCL: now also U$1.12
- net SDA: now also U$1.2
- net VSW: now also L1.1; no longer U$1.1
Routing:
- net +3V3: track 211.7 -> 175.8 mm
- net BATV: track 158.2 -> 135.7 mm
- net N$16: track 4.24 -> 3.00 mm
- net N$1: track 2.50 -> 3.00 mm

Commit message: PCB:
Parts:
- C16, C17: value (none) -> 0.1uF
- moved C16 27.4 mm to (22.7, 7.80)
- moved U$1 25.6 mm to (22.5, 5.00), turned to 180 degrees
- moved C17 25.5 mm to (19.4, 4.80), turned to 270 degrees
Connections:
- net +3V3: now also U$1.10
- net GND: now also U$1.1, U$1.11, U$1.4
Routing:
- net +3V3: track 175.8 -> 243.5 mm, vias 8 -> 9
- net CS_ACCEL: track 22.5 -> 0.00 mm
- net SCL: track 128.7 -> 149.1 mm
- net SDA: track 124.9 -> 142.8 mm, vias 2 -> 3
- net GND: track 3.80 -> 4.93 mm, vias 1 -> 2
- added copper zone on layer 1, net GND
Other:
- board size 45 x 100 mm -> 45 x 98 mm
