File: PCB/CertStack/CertStack.brd (EAGLE design)
At the start: 45 x 98 mm, 57 parts, among them J1 MEM2075-00-140-01-A, Q1 SI2302, Q2 SI2302, Q3 SI2302, Q4 SI2302, Q5 MMBT2222A, T1 DMP3098L-7, U1 TEENSY-32, U2 LT1374CS8-5PBF, U3 SST26VF064B-104V/MN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

Commit message: PCB
Connections:
- removed net CS_ACCEL: U1.15
- net CS_BAR: now also U1.16
- net CS_IMU: now also U1.15
Routing:
- net CS_BAR: track 1.17 -> 33.6 mm
- net CS_IMU: track 0.00 -> 19.3 mm, vias 0 -> 1
- net +3V3: track 243.5 -> 245.6 mm
Changed lines of the file:
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@@
 <wire x1="21.75" y1="7.8" x2="21.75" y2="9.425" width="0.2" layer="1"/>
 <wire x1="21.75" y1="9.425" x2="21.7375" y2="9.4375" width="0.2" layer="1"/>
-<wire x1="19.4" y1="5.75" x2="21.7375" y2="5.75" width="0.2" layer="1"/>
+<wire x1="19.4" y1="5.75" x2="20.5" y2="5.75" width="0.2" layer="1"/>
+<wire x1="20.5" y1="5.75" x2="21.7375" y2="5.75" width="0.2" layer="1"/>
 <wire x1="21.7375" y1="5.75" x2="21.75" y2="5.7625" width="0.2" layer="1"/>
 <wire x1="21.75" y1="5.7625" x2="21.75" y2="6.2" width="0.2" layer="1"/>
@@
 <wire x1="32.3" y1="57.2" x2="29.1" y2="54" width="0.3" layer="16"/>
 <wire x1="28.4" y1="52.9" x2="18.7" y2="52.9" width="0.3" layer="16"/>
-<wire x1="21.7375" y1="4.25" x2="21.7375" y2="5.75" width="0" layer="19" extent="1-1"/>
+<wire x1="21.7375" y1="4.25" x2="21.6875" y2="4.3" width="0.25" layer="1"/>
+<wire x1="21.6875" y1="4.3" x2="21.46538125" y2="4.3" width="0.25" layer="1"/>
+<wire x1="21.46538125" y1="4.3" x2="21" y2="4.76538125" width="0.25" layer="1"/>
+<wire x1="21" y1="5.25" x2="20.5" y2="5.75" width="0.25" layer="1"/>
+<wire x1="21" y1="4.76538125" x2="21" y2="5.25" width="0.25" layer="1"/>
 </signal>
 <signal name="CS_BAR">
@@
 <via x="8.7" y="77.3" extent="1-16" drill="0.35"/>
 <wire x1="7.785" y1="76.775" x2="8.2392625" y2="76.775" width="0.2" layer="1"/>
-<wire x1="8.2392625" y1="76.775" x2="8.7" y2="77.2357375" width="0.2" layer="1"/>
-<wire x1="8.7" y1="77.2357375" x2="8.7" y2="77.3" width="0.2" layer="1"/>
+<wire x1="8.2392625" y1="76.775" x2="8.7642625" y2="77.3" width="0.2" layer="1"/>
+<wire x1="8.7642625" y1="77.3" x2="8.7" y2="77.3" width="0.2" layer="1"/>
+<contactref element="U1" pad="16"/>
+<wire x1="8.7" y1="77.3" x2="13.2" y2="77.3" width="0.25" layer="15"/>
+<wire x1="13.9" y1="78" x2="13.9" y2="78.4" width="0.25" layer="15"/>
+<wire x1="13.9" y1="78.4" x2="14.1" y2="78.6" width="0.25" layer="15"/>
+<wire x1="27.8" y1="79.5" x2="28.7" y2="78.6" width="0.25" layer="15"/>
+<wire x1="28.7" y1="78.6" x2="31.4" y2="78.6" width="0.25" layer="15"/>
+<wire x1="31.4" y1="78.6" x2="32.1" y2="77.9" width="0.25" layer="15"/>
+<wire x1="32.1" y1="77.9" x2="32.1" y2="73.2" width="0.25" layer="15"/>
+<wire x1="32.1" y1="73.2" x2="31.12" y2="72.22" width="0.25" layer="15"/>
+<wire x1="31.12" y1="72.22" x2="30.12" y2="72.22" width="0.25" layer="15"/>
+<wire x1="13.2" y1="77.3" x2="13.9" y2="78" width="0.25" layer="15"/>
+<wire x1="14.1" y1="78.6" x2="26" y2="78.6" width="0.25" layer="15"/>
+<wire x1="26" y1="78.6" x2="26.9" y2="79.5" width="0.25" layer="15"/>
+<wire x1="26.9" y1="79.5" x2="27.8" y2="79.5" width="0.25" layer="15"/>
 </signal>
 <signal name="INT">
@@
 <signal name="CS_IMU">
 <contactref element="U5" pad="5"/>
+<contactref element="U1" pad="15"/>
+<wire x1="21.5" y1="56.665" x2="20.1734" y2="56.665" width="0.25" layer="1"/>
+<wire x1="20.1734" y1="56.665" x2="20.1" y2="56.5916" width="0.25" layer="1"/>
+<via x="20.1" y="56.5916" extent="1-16" drill="0.35"/>
+<wire x1="20.1" y1="56.5916" x2="27.0214" y2="63.513" width="0.25" layer="15"/>
+<wire x1="30.12" y1="68.67725625" x2="30.12" y2="69.68" width="0.25" layer="15"/>
+<wire x1="27.0214" y1="63.513" x2="28.03025625" y2="63.513" width="0.25" layer="15"/>
+<wire x1="29.033" y1="67.59025625" x2="30.12" y2="68.67725625" width="0.25" layer="15"/>
+<wire x1="28.03025625" y1="63.513" x2="29.033" y2="64.51574375" width="0.25" layer="15"/>
+<wire x1="29.033" y1="64.51574375" x2="29.033" y2="67.59025625" width="0.25" layer="15"/>
 </signal>
 <signal name="SCL">
@@
 <contactref element="CAMERA" pad="6"/>
 </signal>
-<signal name="CS_ACCEL">
-<contactref element="U1" pad="15"/>
-</signal>
 <signal name="CS_SD">

Commit message: PCB
Parts:
- R1: value 150 -> 62
- R3: value 15 -> 71.5
- moved BATT-CON 2.00 mm to (33.0, 33.6)
- moved C1 2.00 mm to (39.1, 57.0)
- moved C10 2.00 mm to (27.9, 57.8)
- moved C11 2.00 mm to (25.7, 57.8)
- moved C12 2.00 mm to (26.8, 52.3)
- moved C13 2.00 mm to (25.9, 48.0)
- moved C14 2.00 mm to (28.2, 48.2)
- moved C15 2.00 mm to (2.30, 66.0)
- moved C16 2.00 mm to (22.7, 5.80)
- moved C17 2.00 mm to (19.4, 2.80)
- moved C2 2.00 mm to (27.0, 44.4)
- moved C3 2.00 mm to (27.0, 33.6)
- moved C4 2.00 mm to (27.0, 37.2)
- moved C5 2.00 mm to (27.0, 40.8)
- moved C6 2.00 mm to (7.00, 80.0)
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Connections:
- removed net N$1: R10.1, R11.2
- new net BAT-SENSE: R10.1, R11.2, U1.23
Routing:
- net BAT-SENSE: track 0.00 -> 7.10 mm
- net N$1: track 3.00 -> 0.00 mm
- net +5V: track 160.7 -> 158.6 mm
- net GND: track 4.93 -> 3.93 mm, vias 2 -> 6
- added copper zone on layer 15, net GND
- added copper zone on layer 16, net GND
- added copper zone on layer 2, net GND
Other:
- outline, holes or cut-outs redrawn
