File: PCB/CertStack/CertStack.sch (EAGLE design)
At the start: 42 parts, among them J1 MEM2075-00-140-01-A, Q1 AOD4184A, Q2 AOD4184A, Q3 AOD4184A, Q4 AOD4184A, Q5 MMBT2222A, T1 DMP3098L-7, U2 INVENSENSE_ICM-20608-GINVENSE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, U3 SST26VF064B-104V/MN, U4 LT1374CS8-5PBF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

Commit message: PCB
Parts:
- removed XT1: XT30-RH, mylibrary:XT30-RH
- added BATTERY, SWITCH: (no value), pinhead:PINHD-1X2
- added CAN, I2C: (no value), pinhead:PINHD-1X4
- added GPS, POWER, SPI, TELEM, VTX: (no value), pinhead:PINHD-1X6
- renumbered JP1 to CAMERA
Connections:
- net GND: now also BATTERY.2; no longer XT1.-
- net VCC: now also BATTERY.1; no longer XT1.+
Changed lines of the file:
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@@
 <part name="P+4" library="supply1" library_urn="urn:adsk.eagle:library:371" deviceset="VCC" device=""/>
 <part name="GND16" library="supply1" library_urn="urn:adsk.eagle:library:371" deviceset="GND" device=""/>
-<part name="XT1" library="mylibrary" deviceset="XT30-RH" device=""/>
-<part name="JP1" library="pinhead" library_urn="urn:adsk.eagle:library:325" deviceset="PINHD-1X4" device="" package3d_urn="urn:adsk.eagle:package:22407/2"/>
+<part name="CAMERA" library="pinhead" library_urn="urn:adsk.eagle:library:325" deviceset="PINHD-1X4" device="" package3d_urn="urn:adsk.eagle:package:22407/2"/>
 <part name="GND17" library="supply1" library_urn="urn:adsk.eagle:library:371" deviceset="GND" device=""/>
 <part name="R3" library="rcl" library_urn="urn:adsk.eagle:library:334" deviceset="R-US_" device="R0805" package3d_urn="urn:adsk.eagle:package:23553/2" value="360k"/>
@@
 <part name="R14" library="rcl" library_urn="urn:adsk.eagle:library:334" deviceset="R-US_" device="R0805" package3d_urn="urn:adsk.eagle:package:23553/2" value="100"/>
 <part name="+3V8" library="supply1" library_urn="urn:adsk.eagle:library:371" deviceset="+3V3" device=""/>
+<part name="BATTERY" library="pinhead" library_urn="urn:adsk.eagle:library:325" deviceset="PINHD-1X2" device="" package3d_urn="urn:adsk.eagle:package:22435/2"/>
+<part name="SWITCH" library="pinhead" library_urn="urn:adsk.eagle:library:325" deviceset="PINHD-1X2" device="" package3d_urn="urn:adsk.eagle:package:22435/2"/>
+<part name="VTX" library="pinhead" library_urn="urn:adsk.eagle:library:325" deviceset="PINHD-1X6" device="" package3d_urn="urn:adsk.eagle:package:22472/2"/>
+<part name="GPS" library="pinhead" library_urn="urn:adsk.eagle:library:325" deviceset="PINHD-1X6" device="" package3d_urn="urn:adsk.eagle:package:22472/2"/>
+<part name="TELEM" library="pinhead" library_urn="urn:adsk.eagle:library:325" deviceset="PINHD-1X6" device="" package3d_urn="urn:adsk.eagle:package:22472/2"/>
+<part name="CAN" library="pinhead" library_urn="urn:adsk.eagle:library:325" deviceset="PINHD-1X4" device="" package3d_urn="urn:adsk.eagle:package:22407/2"/>
+<part name="I2C" library="pinhead" library_urn="urn:adsk.eagle:library:325" deviceset="PINHD-1X4" device="" package3d_urn="urn:adsk.eagle:package:22407/2"/>
+<part name="SPI" library="pinhead" library_urn="urn:adsk.eagle:library:325" deviceset="PINHD-1X6" device="" package3d_urn="urn:adsk.eagle:package:22472/2"/>
+<part name="POWER" library="pinhead" library_urn="urn:adsk.eagle:library:325" deviceset="PINHD-1X6" device="" package3d_urn="urn:adsk.eagle:package:22472/2"/>
 </parts>
 <sheets>
@@
 <attribute name="NAME" x="-193.04" y="162.941" size="1.778" layer="95"/>
 </instance>
-<instance part="P+4" gate="VCC" x="-313.69" y="143.51" smashed="yes" rot="R180">
-<attribute name="VALUE" x="-317.754" y="140.97" size="1.778" layer="96"/>
-</instance>
-<instance part="GND16" gate="1" x="-308.61" y="143.51" smashed="yes">
-<attribute name="VALUE" x="-309.372" y="141.224" size="1.778" layer="96"/>
-</instance>
-<instance part="XT1" gate="G$1" x="-311.15" y="158.75" smashed="yes"/>
-<instance part="JP1" gate="A" x="-36.83" y="140.97" smashed="yes">
+<instance part="P+4" gate="VCC" x="-313.69" y="146.05" smashed="yes" rot="R180">
+<attribute name="VALUE" x="-317.754" y="143.51" size="1.778" layer="96"/>
+</instance>
+<instance part="GND16" gate="1" x="-308.61" y="146.05" smashed="yes">
+<attribute name="VALUE" x="-309.372" y="143.764" size="1.778" layer="96"/>
+</instance>
+<instance part="CAMERA" gate="A" x="-36.83" y="140.97" smashed="yes">
 <attribute name="NAME" x="-43.18" y="149.225" size="1.778" layer="95"/>
 <attribute name="VALUE" x="-43.18" y="133.35" size="1.778" layer="96"/>
@@
 <instance part="+3V8" gate="G$1" x="-355.6" y="35.56" smashed="yes">
 <attribute name="VALUE" x="-353.06" y="35.56" size="1.778" layer="96" rot="R90"/>
+</instance>
+<instance part="BATTERY" gate="G$1" x="-309.88" y="157.48" smashed="yes" rot="R90">
+<attribute name="NAME" x="-315.595" y="151.13" size="1.778" layer="95" rot="R90"/>
+<attribute name="VALUE" x="-304.8" y="151.13" size="1.778" layer="96" rot="R90"/>
+</instance>
+<instance part="SWITCH" gate="G$1" x="-294.64" y="157.48" smashed="yes" rot="R90">
+<attribute name="NAME" x="-300.355" y="151.13" size="1.778" layer="95" rot="R90"/>
+<attribute name="VALUE" x="-289.56" y="151.13" size="1.778" layer="96" rot="R90"/>
+</instance>
+<instance part="VTX" gate="A" x="-17.78" y="142.24" smashed="yes">
+<attribute name="NAME" x="-24.13" y="153.035" size="1.778" layer="95"/>
+<attribute name="VALUE" x="-24.13" y="132.08" size="1.778" layer="96"/>
+</instance>
+<instance part="GPS" gate="A" x="-2.54" y="142.24" smashed="yes">
+<attribute name="NAME" x="-8.89" y="153.035" size="1.778" layer="95"/>
+<attribute name="VALUE" x="-8.89" y="132.08" size="1.778" layer="96"/>
+</instance>
+<instance part="TELEM" gate="A" x="12.7" y="142.24" smashed="yes">
+<attribute name="NAME" x="6.35" y="153.035" size="1.778" layer="95"/>
+<attribute name="VALUE" x="6.35" y="132.08" size="1.778" layer="96"/>
+</instance>
+<instance part="CAN" gate="A" x="-36.83" y="171.45" smashed="yes">
+<attribute name="NAME" x="-43.18" y="179.705" size="1.778" layer="95"/>
+<attribute name="VALUE" x="-43.18" y="163.83" size="1.778" layer="96"/>
+</instance>
+<instance part="I2C" gate="A" x="-6.35" y="171.45" smashed="yes">
+<attribute name="NAME" x="-12.7" y="179.705" size="1.778" layer="95"/>
+<attribute name="VALUE" x="-12.7" y="163.83" size="1.778" layer="96"/>
+</instance>
+<instance part="SPI" gate="A" x="-22.86" y="172.72" smashed="yes">
+<attribute name="NAME" x="-29.21" y="183.515" size="1.778" layer="95"/>
+<attribute name="VALUE" x="-29.21" y="162.56" size="1.778" layer="96"/>
+</instance>
+<instance part="POWER" gate="A" x="25.4" y="172.72" smashed="yes">
+<attribute name="NAME" x="19.05" y="183.515" size="1.778" layer="95"/>
+<attribute name="VALUE" x="19.05" y="162.56" size="1.778" layer="96"/>
 </instance>
 </instances>
@@
 </segment>
 <segment>
-<pinref part="GND16" gate="1" pin="GND"/>
-<wire x1="-308.61" y1="148.59" x2="-308.61" y2="146.05" width="0.1524" layer="91"/>
-<pinref part="XT1" gate="G$1" pin="-"/>
-</segment>
-<segment>
-<pinref part="JP1" gate="A" pin="2"/>
+<pinref part="CAMERA" gate="A" pin="2"/>
 <wire x1="-39.37" y1="143.51" x2="-49.53" y2="143.51" width="0.1524" layer="91"/>
 <wire x1="-49.53" y1="143.51" x2="-49.53" y2="146.05" width="0.1524" layer="91"/>
@@
 <pinref part="LED3" gate="G$1" pin="C"/>
 <wire x1="-340.36" y1="137.16" x2="-340.36" y2="139.7" width="0.1524" layer="91"/>
+</segment>
+<segment>
+<pinref part="GND16" gate="1" pin="GND"/>
+<pinref part="BATTERY" gate="G$1" pin="2"/>
+<wire x1="-308.61" y1="148.59" x2="-308.61" y2="154.94" width="0.1524" layer="91"/>
+<wire x1="-308.61" y1="154.94" x2="-309.88" y2="154.94" width="0.1524" layer="91"/>
 </segment>
 </net>
@@
 <net name="VCC" class="0">
 <segment>
-<pinref part="P+4" gate="VCC" pin="VCC"/>
-<wire x1="-313.69" y1="148.59" x2="-313.69" y2="146.05" width="0.1524" layer="91"/>
-<pinref part="XT1" gate="G$1" pin="+"/>
-</segment>
-<segment>
 <pinref part="X3" gate="-1" pin="K"/>
 <wire x1="-196.85" y1="168.91" x2="-204.47" y2="168.91" width="0.1524" layer="91"/>
@@
 <pinref part="P+3" gate="VCC" pin="VCC"/>
 </segment>
+<segment>
+<pinref part="P+4" gate="VCC" pin="VCC"/>
+<pinref part="BATTERY" gate="G$1" pin="1"/>
+<wire x1="-313.69" y1="148.59" x2="-313.69" y2="154.94" width="0.1524" layer="91"/>
+<wire x1="-313.69" y1="154.94" x2="-312.42" y2="154.94" width="0.1524" layer="91"/>
+</segment>
 </net>
 <net name="N$2" class="0">
 <segment>
-<pinref part="JP1" gate="A" pin="1"/>
+<pinref part="CAMERA" gate="A" pin="1"/>
 <wire x1="-39.37" y1="146.05" x2="-46.99" y2="146.05" width="0.1524" layer="91"/>
 <wire x1="-46.99" y1="146.05" x2="-46.99" y2="151.13" width="0.1524" layer="91"/>
@@
 <net name="VID-IN" class="0">
 <segment>
-<pinref part="JP1" gate="A" pin="3"/>
+<pinref part="CAMERA" gate="A" pin="3"/>
 <wire x1="-39.37" y1="140.97" x2="-49.53" y2="140.97" width="0.1524" layer="91"/>
 <wire x1="-49.53" y1="140.97" x2="-49.53" y2="138.43" width="0.1524" layer="91"/>
@@
 <net name="CC" class="0">
 <segment>
-<pinref part="JP1" gate="A" pin="4"/>
+<pinref part="CAMERA" gate="A" pin="4"/>
 <wire x1="-39.37" y1="138.43" x2="-46.99" y2="138.43" width="0.1524" layer="91"/>
 <wire x1="-46.99" y1="138.43" x2="-46.99" y2="133.35" width="0.1524" layer="91"/>

Commit message: PCB
Parts:
- removed R21: 360k, rcl:R-US_R0805
- removed R22: 51k, rcl:R-US_R0805
- removed R23, R5, R6, R9: 10k, rcl:R-US_R0805
- removed X1, X2, X3, X4: TERMINAL-BLOCK-3.5MM-2-PIN-LONG-PAD, Rembrandt Electronics - Terminal Block 3-5mm v1-0:TERMINAL-BLOCK-3.5MM-2-PIN-LONG-PAD
- added R1, R2: 10k, rcl:R-US_R0805
- Q1, Q2, Q3, Q4: value AOD4184A -> SI2302; device AOD4184A:AOD4184A -> SI2302:SI2302
- R3: value 360k -> 10k
- R4: value 51k -> 10k
Connections:
- removed net CE: U3.CE#
- removed net PY1_D: R21.1, R22.2
- removed net PY1_F: Q3.G, R23.2
- removed net PY2_D: R3.1, R4.2
- removed net PY2_F: Q1.G, R5.2
- removed net PY3_F: Q2.G, R6.2
- removed net PY4_F: Q4.G, R9.2
- removed net SDI: BMP384_1.4, U2.SDA/SDI
- removed net SDO: BMP384_1.5, U2.AD0/SDO
- new net BATV: R14.2
- new net CS_FLASH: U$1.2, U3.CE#
- new net N$1: Q1.G, R1.2
- new net N$10: Q4.G, R4.2
- new net N$11: Q4.D
- new net N$8: Q3.G, R3.2
- net +3V3: no longer BMP384_1.3, C2.2
- net +5V: no longer X2-1.K, X4-1.K
- net CS_BAR: now also U$1.6
- net GND: now also BMP384_1.3, C2.2, R1.1, R2.1, R3.1; no longer R22.1, R23.1, R5.1, R6.1, R9.1
- net MISO: now also BMP384_1.5, U2.AD0/SDO
- net MOSI: now also BMP384_1.4, U2.SDA/SDI
- net N$3: no longer R3.2, X1-2.K
- net N$4: now also Q2.G, R2.2; no longer Q4.D, X4-2.K
- net N$5: no longer X2-2.K
- net N$9: no longer R21.2, X3-2.K
- net VCC: no longer X1-1.K, X3-1.K
Other:
- moved on the sheet: R3, R4

Commit message: PCB
Parts:
- removed CAN, I2C: (no value), pinhead:PINHD-1X4
- removed SPI: (no value), pinhead:PINHD-1X6
- removed SWITCH: (no value), pinhead:PINHD-1X2
- added DATA: (no value), mylibrary:JST-PH-6
- CAMERA: device pinhead:PINHD-1X4 -> mylibrary:JST-PH-6
- GPS, POWER, TELEM, VTX: device pinhead:PINHD-1X6 -> mylibrary:JST-PH-6
Connections:
- net N$11 renamed FET4
- net N$5 renamed FET3
- removed net VID-IN: CAMERA.3
- new net CANH: DATA.6
- new net CANL: DATA.5
- new net FET1: Q1.D, TELEM.1
- new net FET2: CAMERA.1, Q3.D, VTX.1
- new net GPS_RX: GPS.3
- new net GPS_TX: GPS.4
- new net N$11: GPS.6
- new net SW+: POWER.5
- new net SW-: POWER.6
- new net TELEM_RX: TELEM.3
- new net TELEM_TX: TELEM.4
- new net VIDEO: CAMERA.3, VTX.3
- new net VTX_RX: VTX.4
- new net VTX_TX: VTX.5
- net +3V3: now also DATA.2, GPS.2, POWER.2
- net +5V: now also POWER.3, TELEM.2
- net BATV: now also CAMERA.2, POWER.4, VTX.2
- net GND: now also DATA.1, GPS.1, POWER.1, TELEM.6, VTX.6; no longer CAMERA.2
- net N$2: now also CAMERA.5; no longer CAMERA.1
- net N$3: now also CAMERA.6; no longer Q1.D
- net N$9: now also GPS.5; no longer Q3.D
- net SCL: now also DATA.3
- net SDA: now also DATA.4

Commit message: PCB
Connections:
- removed net N$1: Q1.G, R1.2
- removed net N$10: Q4.G, R4.2
- removed net N$4: Q2.G, R2.2
- removed net N$8: Q3.G, R3.2
- new net F1_TRIG: Q1.G, R1.2, U$1.3
- new net F2_TRIG: Q2.G, R2.2, U$1.4
- new net F3_TRIG: Q3.G, R3.2, U$1.5
- new net F4_TRIG: Q4.G, R4.2, U$1.6
- net CS_BAR: no longer U$1.6
- net FET2: now also Q2.D; no longer Q3.D
- net FET3: now also Q3.D; no longer Q2.D
- net GPS_RX: now also U$1.9
- net GPS_TX: now also U$1.10
- net TELEM_RX: now also U$1.0
- net TELEM_TX: now also U$1.1
- net VTX_RX: now also U$1.7
- net VTX_TX: now also U$1.8
Other:
- moved on the sheet: Q2, Q3, Q4, R2, R3, R4

Commit message: PCB
Parts:
- removed BATTERY: (no value), pinhead:PINHD-1X2
- added U$2: PWR-AWG18, mylibrary:PWR-AWG18
Connections:
- new net CS_ACCEL: U$1.15
- new net CS_SD: U$1.14
- net CS-SD: no longer U$1.14
- net GND: now also U$2.-; no longer BATTERY.2
- net VCC: now also U$2.+; no longer BATTERY.1
Changed lines of the file:
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@@
 <part name="+3V11" library="supply1" library_urn="urn:adsk.eagle:library:371" deviceset="+3V3" device=""/>
 <part name="GND24" library="supply1" library_urn="urn:adsk.eagle:library:371" deviceset="GND" device=""/>
-<part name="P+4" library="supply1" library_urn="urn:adsk.eagle:library:371" deviceset="VCC" device=""/>
-<part name="GND16" library="supply1" library_urn="urn:adsk.eagle:library:371" deviceset="GND" device=""/>
 <part name="LS1" library="mylibrary" deviceset="CMT-8540S" device=""/>
 <part name="GND26" library="supply1" library_urn="urn:adsk.eagle:library:371" deviceset="GND" device=""/>
@@
 <part name="R14" library="rcl" library_urn="urn:adsk.eagle:library:334" deviceset="R-US_" device="R0805" package3d_urn="urn:adsk.eagle:package:23553/2" value="100"/>
 <part name="+3V8" library="supply1" library_urn="urn:adsk.eagle:library:371" deviceset="+3V3" device=""/>
-<part name="BATTERY" library="pinhead" library_urn="urn:adsk.eagle:library:325" deviceset="PINHD-1X2" device="" package3d_urn="urn:adsk.eagle:package:22435/2"/>
 <part name="GND3" library="supply1" library_urn="urn:adsk.eagle:library:371" deviceset="GND" device=""/>
 <part name="Q1" library="SI2302" deviceset="SI2302" device=""/>
@@
 <part name="+3V3" library="supply1" library_urn="urn:adsk.eagle:library:371" deviceset="+3V3" device=""/>
 <part name="+3V10" library="supply1" library_urn="urn:adsk.eagle:library:371" deviceset="+3V3" device=""/>
+<part name="U$2" library="mylibrary" deviceset="PWR-AWG18" device=""/>
+<part name="P+1" library="supply1" library_urn="urn:adsk.eagle:library:371" deviceset="VCC" device=""/>
+<part name="GND25" library="supply1" library_urn="urn:adsk.eagle:library:371" deviceset="GND" device=""/>
 </parts>
 <sheets>
@@
 <attribute name="VALUE" x="-260.35" y="-24.13" size="1.778" layer="96"/>
 </instance>
-<instance part="P+4" gate="VCC" x="-313.69" y="146.05" smashed="yes" rot="R180">
-<attribute name="VALUE" x="-317.754" y="143.51" size="1.778" layer="96"/>
-</instance>
-<instance part="GND16" gate="1" x="-308.61" y="146.05" smashed="yes">
-<attribute name="VALUE" x="-309.372" y="143.764" size="1.778" layer="96"/>
-</instance>
 <instance part="LS1" gate="G$1" x="-375.92" y="160.02" smashed="yes"/>
 <instance part="GND26" gate="1" x="-373.38" y="134.62" smashed="yes">
@@
 <attribute name="VALUE" x="-353.06" y="35.56" size="1.778" layer="96" rot="R90"/>
 </instance>
-<instance part="BATTERY" gate="G$1" x="-309.88" y="157.48" smashed="yes" rot="R90">
-<attribute name="NAME" x="-315.595" y="151.13" size="1.778" layer="95" rot="R90"/>
-<attribute name="VALUE" x="-304.8" y="151.13" size="1.778" layer="96" rot="R90"/>
-</instance>
 <instance part="GND3" gate="1" x="-411.48" y="40.64" smashed="yes" rot="R270">
 <attribute name="VALUE" x="-414.02" y="43.18" size="1.778" layer="96" rot="R270"/>
@@
 <instance part="+3V10" gate="G$1" x="-17.78" y="157.48" smashed="yes" rot="R180">
 <attribute name="VALUE" x="-15.24" y="162.56" size="1.778" layer="96" rot="R270"/>
+</instance>
+<instance part="U$2" gate="G$1" x="-292.1" y="152.4" smashed="yes"/>
+<instance part="P+1" gate="VCC" x="-299.72" y="160.02" smashed="yes">
+<attribute name="VALUE" x="-295.656" y="162.56" size="1.778" layer="96" rot="R180"/>
+</instance>
+<instance part="GND25" gate="1" x="-299.72" y="144.78" smashed="yes">
+<attribute name="VALUE" x="-300.482" y="142.494" size="1.778" layer="96"/>
 </instance>
 </instances>
@@
 </segment>
 <segment>
-<pinref part="GND16" gate="1" pin="GND"/>
-<pinref part="BATTERY" gate="G$1" pin="2"/>
-<wire x1="-308.61" y1="148.59" x2="-308.61" y2="154.94" width="0.1524" layer="91"/>
-<wire x1="-308.61" y1="154.94" x2="-309.88" y2="154.94" width="0.1524" layer="91"/>
-</segment>
-<segment>
 <pinref part="GND2" gate="1" pin="GND"/>
 <pinref part="C2" gate="G$1" pin="2"/>
@@
 <wire x1="-45.72" y1="213.36" x2="-45.72" y2="210.82" width="0.1524" layer="91"/>
 <pinref part="GND17" gate="1" pin="GND"/>
+</segment>
+<segment>
+<pinref part="U$2" gate="G$1" pin="-"/>
+<pinref part="GND25" gate="1" pin="GND"/>
+<wire x1="-297.18" y1="149.86" x2="-299.72" y2="149.86" width="0.1524" layer="91"/>
+<wire x1="-299.72" y1="149.86" x2="-299.72" y2="147.32" width="0.1524" layer="91"/>
 </segment>
 </net>
@@
 <label x="-303.53" y="-19.05" size="1.778" layer="95" rot="R180" xref="yes"/>
 </segment>
-<segment>
-<pinref part="U$1" gate="G$1" pin="14"/>
-<wire x1="-363.22" y1="-20.32" x2="-350.52" y2="-20.32" width="0.1524" layer="91"/>
-<label x="-350.52" y="-20.32" size="1.778" layer="95" xref="yes"/>
-</segment>
 </net>
 <net name="VCC" class="0">
 <segment>
-<pinref part="P+4" gate="VCC" pin="VCC"/>
-<pinref part="BATTERY" gate="G$1" pin="1"/>
-<wire x1="-313.69" y1="148.59" x2="-313.69" y2="154.94" width="0.1524" layer="91"/>
-<wire x1="-313.69" y1="154.94" x2="-312.42" y2="154.94" width="0.1524" layer="91"/>
+<pinref part="U$2" gate="G$1" pin="+"/>
+<pinref part="P+1" gate="VCC" pin="VCC"/>
+<wire x1="-297.18" y1="154.94" x2="-299.72" y2="154.94" width="0.1524" layer="91"/>
+<wire x1="-299.72" y1="154.94" x2="-299.72" y2="157.48" width="0.1524" layer="91"/>
 </segment>
 </net>
@@
 </segment>
 </net>
+<net name="CS_ACCEL" class="0">
+<segment>
+<pinref part="U$1" gate="G$1" pin="15"/>
+<wire x1="-363.22" y1="-15.24" x2="-350.52" y2="-15.24" width="0.1524" layer="91"/>
+<label x="-350.52" y="-15.24" size="1.778" layer="95" xref="yes"/>
+</segment>
+</net>
+<net name="CS_SD" class="0">
+<segment>
+<pinref part="U$1" gate="G$1" pin="14"/>
+<wire x1="-363.22" y1="-20.32" x2="-350.52" y2="-20.32" width="0.1524" layer="91"/>
+<label x="-350.52" y="-20.32" size="1.778" layer="95" xref="yes"/>
+</segment>
+</net>

Commit message: PCB
Parts:
- removed U4: LT1374CS8-5PBF, LT1374CS8-5PBF:LT1374CS8-5PBF
- added C10, C11: 10uF, SparkFun-Capacitors:10UF-1206-6.3V-20%
- added C4: (no value), rcl:C-USC0805
- added CC: 1.5nF, rcl:C-USC0805
- added D1: 1N4004, diode:1N4004
- added D2: 30V 100mA, diode:1N821
- added L1: 5 uH, ngspice-simulation:L
- added U1: LT1374CS8-5PBF, LT1374CS8-5PBF:LT1374CS8-5PBF
Connections:
- removed net SW+: POWER.5
- removed net SW-: POWER.6
- removed net V_BAT: U4.VIN
- new net BOOST: C4.2, D2.A, U1.BOOST
- new net OUT: D2.C, L1.2
- new net SENSE: D1.C, U1.BIAS, U1.FB/SENSE
- new net SHDN: POWER.6, U1.SYNC/*SHDN
- new net VC: CC.1, U1.VC
- new net VSW: C4.1, L1.1, U1.VSW
- net BATV: now also C10.1, C11.1, U1.VIN
- net GND: now also C10.2, C11.2, CC.2, D1.A, POWER.5, U1.FGND; no longer U4.FGND

Commit message: PCB
Parts:
- removed D2: 30V 100mA, diode:1N821
- added U$3: DO-214AB, DO-214AB:DO-214AB
Connections:
- net BOOST: no longer D2.A
- net OUT: no longer D2.C
Changed lines of the file:
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@@
 <part name="U1" library="LT1374CS8-5PBF" deviceset="LT1374CS8-5PBF" device=""/>
 <part name="GND30" library="supply1" library_urn="urn:adsk.eagle:library:371" deviceset="GND" device=""/>
-<part name="D2" library="diode" library_urn="urn:adsk.eagle:library:210" deviceset="1N821" device="" package3d_urn="urn:adsk.eagle:package:43342/1" value="30V 100mA"/>
 <part name="C4" library="rcl" library_urn="urn:adsk.eagle:library:334" deviceset="C-US" device="C0805" package3d_urn="urn:adsk.eagle:package:23617/2"/>
 <part name="L1" library="ngspice-simulation" library_urn="urn:adsk.eagle:library:527439" deviceset="L" device="" value="5 uH"/>
@@
 <part name="GND36" library="supply1" library_urn="urn:adsk.eagle:library:371" deviceset="GND" device=""/>
 <part name="GND16" library="supply1" library_urn="urn:adsk.eagle:library:371" deviceset="GND" device=""/>
+<part name="U$3" library="DO-214AB" deviceset="DO-214AB" device=""/>
 </parts>
 <sheets>
@@
 <attribute name="VALUE" x="-254" y="63.5" size="1.778" layer="96" rot="R270"/>
 </instance>
-<instance part="D2" gate="1" x="-238.76" y="45.72" smashed="yes">
-<attribute name="NAME" x="-240.538" y="47.625" size="1.778" layer="95"/>
-<attribute name="VALUE" x="-240.538" y="42.291" size="1.778" layer="96"/>
-</instance>
 <instance part="C4" gate="G$1" x="-208.28" y="45.72" smashed="yes" rot="R270">
 <attribute name="NAME" x="-207.645" y="44.704" size="1.778" layer="95" rot="R270"/>
@@
 <attribute name="VALUE" x="-5.08" y="205.74" size="1.778" layer="96"/>
 </instance>
+<instance part="U$3" gate="G$1" x="-142.24" y="58.42" smashed="yes"/>
 </instances>
 <busses>
@@
 </segment>
 <segment>
-<wire x1="-246.38" y1="45.72" x2="-241.3" y2="45.72" width="0.1524" layer="91"/>
-<label x="-251.46" y="45.72" size="1.778" layer="95"/>
-<pinref part="D2" gate="1" pin="A"/>
-</segment>
-<segment>
 <wire x1="-218.44" y1="45.72" x2="-213.36" y2="45.72" width="0.1524" layer="91"/>
 <pinref part="C4" gate="G$1" pin="2"/>
@@
 <net name="OUT" class="0">
 <segment>
-<pinref part="D2" gate="1" pin="C"/>
-<wire x1="-236.22" y1="45.72" x2="-228.6" y2="45.72" width="0.1524" layer="91"/>
-<label x="-233.68" y="45.72" size="1.778" layer="95"/>
-</segment>
-<segment>
 <pinref part="L1" gate="G$1" pin="2"/>

Commit message: PCB
Parts:
- removed U$3: DO-214AB, DO-214AB:DO-214AB
- added C3: (no value), rcl:C-USC0805
- added D2: DO-214AB, DO-214AB:DO-214AB
- D1: value 1N4004 -> PMEG4020ETP,115; device diode:1N4004 -> PMEG4020ETP_115:PMEG4020ETP,115
Connections:
- removed net SENSE: D1.C, U1.BIAS, U1.FB/SENSE
- net BOOST: now also D2.OUT
- net GND: now also C3.2
- net OUT: now also C3.1, D2.IN, U1.BIAS, U1.FB/SENSE
- net VSW: now also D1.K
Other:
- moved on the sheet: C10, C11, C4, CC, L1, U1
