File: PCB/CertStack/CertStack.sch (EAGLE design)
At the start: 47 parts, among them J1 MEM2075-00-140-01-A, Q1 SI2302, Q2 SI2302, Q3 SI2302, Q4 SI2302, Q5 MMBT2222A, T1 DMP3098L-7, U1 LT1374CS8-5PBF, U2 INVENSENSE_ICM-20608-GINVENSE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, U3 SST26VF064B-104V/MN

Commit message: PCB
Parts:
- removed C3: (no value), rcl:C-USC0805
- added C12: T491X106K050AT, T491X106K050AT:T491X106K050AT
Connections:
- net GND: now also C12.2; no longer C3.2
- net OUT: now also C12.1; no longer C3.1
Changed lines of the file:
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@@
 <part name="D2" library="DO-214AB" deviceset="DO-214AB" device=""/>
 <part name="D1" library="PMEG4020ETP_115" deviceset="PMEG4020ETP,115" device=""/>
-<part name="C3" library="rcl" library_urn="urn:adsk.eagle:library:334" deviceset="C-US" device="C0805" package3d_urn="urn:adsk.eagle:package:23617/2"/>
+<part name="C12" library="T491X106K050AT" deviceset="T491X106K050AT" device=""/>
 </parts>
 <sheets>
@@
 <attribute name="NAME" x="-162.56" y="30.48" size="1.778" layer="95" rot="R90"/>
 </instance>
-<instance part="C3" gate="G$1" x="-134.62" y="38.1" smashed="yes">
-<attribute name="NAME" x="-133.604" y="38.735" size="1.778" layer="95"/>
-<attribute name="VALUE" x="-133.604" y="33.909" size="1.778" layer="96"/>
+<instance part="C12" gate="G$1" x="-134.62" y="35.56" smashed="yes" rot="R90">
+<attribute name="NAME" x="-138.43" y="35.56" size="1.778" layer="95" rot="R90"/>
 </instance>
 </instances>
@@
 <pinref part="CC" gate="G$1" pin="2"/>
 <wire x1="-167.64" y1="33.02" x2="-167.64" y2="27.94" width="0.1524" layer="91"/>
-<pinref part="C3" gate="G$1" pin="2"/>
 <wire x1="-134.62" y1="33.02" x2="-134.62" y2="27.94" width="0.1524" layer="91"/>
 <wire x1="-134.62" y1="27.94" x2="-160.02" y2="27.94" width="0.1524" layer="91"/>
@@
 <wire x1="-160.02" y1="30.48" x2="-160.02" y2="27.94" width="0.1524" layer="91"/>
 <junction x="-160.02" y="27.94"/>
+<pinref part="C12" gate="G$1" pin="2"/>
 </segment>
 </net>
@@
 <wire x1="-172.72" y1="43.18" x2="-177.8" y2="43.18" width="0.1524" layer="91"/>
 <label x="-177.8" y="43.18" size="1.778" layer="95" rot="R180" xref="yes"/>
-<pinref part="C3" gate="G$1" pin="1"/>
 <wire x1="-172.72" y1="45.72" x2="-134.62" y2="45.72" width="0.1524" layer="91"/>
 <wire x1="-134.62" y1="45.72" x2="-134.62" y2="40.64" width="0.1524" layer="91"/>
@@
 <wire x1="-134.62" y1="45.72" x2="-134.62" y2="53.34" width="0.1524" layer="91"/>
 <junction x="-134.62" y="45.72"/>
-</segment>
-<segment>
+<pinref part="C12" gate="G$1" pin="1"/>
+</segment>
+<segment>

Commit message: PCB
Parts:
- removed BMP384_1: BMP384, PQFN45P200X200X100-10N:BMP384
- removed R10, R11: 15, rcl:R-US_R0805
- removed R14: 100, rcl:R-US_R0805
- removed U$1: TEENSY-32, mylibrary:TEENSY-32
- removed U$2: PWR-AWG18, mylibrary:PWR-AWG18
- added BATT-CON: PWR-AWG18, mylibrary:PWR-AWG18
- added R5: 100, rcl:R-US_R0805
- added R6, R9: 10k, rcl:R-US_R0805
- added U4: BMP384, PQFN45P200X200X100-10N:BMP384
- added U5: INVENSENSE_ICM-20608-GINVENSENSE_ICM-20608-G_0_0, InvenSense - ICM-20608-G:INVENSENSE_ICM-20608-GINVENSENSE_ICM-20608-G_0_0
- R1: value 10k -> 150
- R2, R3: value 10k -> 15
- R4: value 10k -> 1k
- R7: value 1k -> 10k
- R8: value 150 -> 10k
- U1: value LT1374CS8-5PBF -> TEENSY-32; device LT1374CS8-5PBF:LT1374CS8-5PBF -> mylibrary:TEENSY-32
- U2: value INVENSENSE_ICM-20608-GINVENSENSE_ICM-20608-G_0_0 -> LT1374CS8-5PBF; device InvenSense - ICM-20608-G:INVENSENSE_ICM-20608-GINVENSENSE_ICM-20608-G_0_0 -> LT1374CS8-5PBF:LT1374CS8-5PBF
Connections:
- net +3V3: now also R1.2, U1.3V3-1, U4.1, U4.10, U5.VDD, U5.VDDIO; no longer BMP384_1.1, BMP384_1.10, R8.2, U$1.3V3-1, U2.VDD, U2.VDDIO
- net BATV: now also R5.2, U2.VIN; no longer R14.2, U1.VIN
- net BOOST: now also U2.BOOST; no longer U1.BOOST
- net BUZZER: now also R4.2, U1.17; no longer R7.2, U$1.17
- net CS_ACCEL: now also U1.15; no longer U$1.15
- net CS_BAR: now also U4.6; no longer BMP384_1.6
- net CS_FLASH: now also U1.2; no longer U$1.2
- net CS_IMU: now also U5.CS; no longer U2.CS
- net CS_SD: now also U1.14; no longer U$1.14
- net F1_TRIG: now also R6.2, U1.3; no longer R1.2, U$1.3
- net F2_TRIG: now also R7.2, U1.4; no longer R2.2, U$1.4
- net F3_TRIG: now also R8.2, U1.5; no longer R3.2, U$1.5
- net F4_TRIG: now also R9.2, U1.6; no longer R4.2, U$1.6
- net GND: now also BATT-CON.-, R6.1, R7.1, R8.1, R9.1, U1.GND1, U1.GND3, U2.FGND, U4.3, U4.8, U4.9, U5.1_RESERVED, U5.2_RESERVED, U5.3_RESERVED, U5.4_RESERVED, U5.5_RESERVED, U5.6_RESERVED, U5.FSYNC, U5.GND; no longer BMP384_1.3, BMP384_1.8, BMP384_1.9, R1.1, R2.1, R3.1, R4.1, U$1.GND1, U$1.GND3, U$2.-, U1.FGND, U2.1_RESERVED, U2.2_RESERVED, U2.3_RESERVED, U2.4_RESERVED, U2.5_RESERVED, U2.6_RESERVED, U2.FSYNC, U2.GND
- net GPS_RX: now also U1.9; no longer U$1.9
- net GPS_TX: now also U1.10; no longer U$1.10
- net INT: now also U4.7; no longer BMP384_1.7
- net LED-ER: now also R3.2, U1.20; no longer R11.2, U$1.20
- net LED-HB: now also R2.2, U1.21; no longer R10.2, U$1.21
- net MISO: now also U1.12, U4.5, U5.AD0/SDO; no longer BMP384_1.5, U$1.12, U2.AD0/SDO
- net MOSI: now also U1.11, U4.4, U5.SDA/SDI; no longer BMP384_1.4, U$1.11, U2.SDA/SDI
- net N$12: now also R5.1; no longer R14.1
- net N$16: now also R1.1; no longer R8.1
- net N$17: now also R2.1; no longer R10.1
- net N$22: now also R4.1; no longer R7.1
- net N$6: now also R3.1; no longer R11.1
- net N$7: now also U5.REGOUT; no longer U2.REGOUT
- net OUT: now also U2.BIAS, U2.FB/SENSE; no longer U1.BIAS, U1.FB/SENSE
- net SCK: now also U1.13, U4.2, U5.SCL/SCLK; no longer BMP384_1.2, U$1.13, U2.SCL/SCLK
- net SCL: now also U1.19; no longer U$1.19
- net SDA: now also U1.18; no longer U$1.18
- net SHDN: now also U2.SYNC/*SHDN; no longer U1.SYNC/*SHDN
- net TELEM_RX: now also U1.0; no longer U$1.0
- net TELEM_TX: now also U1.1; no longer U$1.1
- net VBUS: now also U1.VIN; no longer U$1.VIN
- net VC: now also U2.VC; no longer U1.VC
- net VCC: now also BATT-CON.+; no longer U$2.+
- net VSW: now also U2.VSW; no longer U1.VSW
- net VTX_RX: now also U1.7; no longer U$1.7
- net VTX_TX: now also U1.8; no longer U$1.8
Other:
- note added: "Barometer"
- note added: "Flash"
- note added: "I/O"
- note added: "IMU"
- note added: "Power FETs"
- note added: "Power Supply"
- note added: "Status Indicators"
- moved on the sheet: C1, C10, C11, C12, C2, C4, C5, C6, C7, C8, C9, CAMERA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

Commit message: PCB
Parts:
- removed CC: 1.5nF, rcl:C-USC0805
- removed L1: 5 uH, ngspice-simulation:L
- added C3: 10uF, SparkFun-Capacitors:10UF-1206-6.3V-20%
- added U$1: IHLP3232DZER6R8M11, mylibrary:IHLP3232DZER6R8M11
- C1: value (none) -> T491X106K050AT; device rcl:C-USC0805 -> T491X106K050AT:T491X106K050AT
- C10: value 10uF -> 2.2uF; device SparkFun-Capacitors:10UF-1206-6.3V-20% -> rcl:C-USC0805
- C11: value 10uF -> 10nF; device SparkFun-Capacitors:10UF-1206-6.3V-20% -> rcl:C-USC0805
- C12: value T491X106K050AT -> 0.47uF; device T491X106K050AT:T491X106K050AT -> rcl:C-USC0805
- C4: value (none) -> 10uF; device rcl:C-USC0805 -> SparkFun-Capacitors:10UF-1206-6.3V-20%
- C5: value 2.2uF -> 1.5nF
- C6: value 0.1uF -> 100nF
- C7: value 10nF -> (none)
- C8: value 0.47uF -> (none)
- C9: value 100nF -> 0.1uF
Connections:
- removed net VCC: BATT-CON.+
- net +3V3: now also C10.1, C11.1, C8.1; no longer C1.1, C2.1, C5.1
- net BATV: now also BATT-CON.+, C3.1, C4.1; no longer C10.1, C11.1
- net BOOST: now also C2.2; no longer C4.2
- net GND: now also C3.2, C4.2; no longer C2.2, CC.2
- net N$7: now also C12.1; no longer C8.1
- net OUT: now also C1.1, U$1.2; no longer C12.1, L1.2
- net VC: now also C5.1; no longer CC.1
- net VSW: now also C2.1, U$1.1; no longer C4.1, L1.1
Other:
- moved on the sheet: C1, C10, C11, C12, C2, C4, C5, C6, C7, C8, C9

Commit message: PCB. Big changes.
Parts:
- added R10, R11: ??, rcl:R-US_R0805
Connections:
- new net N$1: R10.1, R11.2
- net BATV: now also R10.2
- net GND: now also R11.1
Changed lines of the file:
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@@
 <part name="C1" library="T491X106K050AT" deviceset="T491X106K050AT" device=""/>
 <part name="U$1" library="mylibrary" deviceset="IHLP3232DZER6R8M11" device=""/>
+<part name="R10" library="rcl" library_urn="urn:adsk.eagle:library:334" deviceset="R-US_" device="R0805" package3d_urn="urn:adsk.eagle:package:23553/2" value="??"/>
+<part name="R11" library="rcl" library_urn="urn:adsk.eagle:library:334" deviceset="R-US_" device="R0805" package3d_urn="urn:adsk.eagle:package:23553/2" value="??"/>
+<part name="GND37" library="supply1" library_urn="urn:adsk.eagle:library:371" deviceset="GND" device=""/>
 </parts>
 <sheets>
@@
 </instance>
 <instance part="U$1" gate="G$1" x="-114.3" y="116.84" smashed="yes"/>
+<instance part="R10" gate="G$1" x="-271.78" y="106.68" smashed="yes" rot="R90">
+<attribute name="NAME" x="-273.2786" y="102.87" size="1.778" layer="95" rot="R90"/>
+<attribute name="VALUE" x="-268.478" y="102.87" size="1.778" layer="96" rot="R90"/>
+</instance>
+<instance part="R11" gate="G$1" x="-271.78" y="91.44" smashed="yes" rot="R90">
+<attribute name="NAME" x="-273.2786" y="87.63" size="1.778" layer="95" rot="R90"/>
+<attribute name="VALUE" x="-268.478" y="87.63" size="1.778" layer="96" rot="R90"/>
+</instance>
+<instance part="GND37" gate="1" x="-271.78" y="78.74" smashed="yes">
+<attribute name="VALUE" x="-274.32" y="76.2" size="1.778" layer="96"/>
+</instance>
 </instances>
 <busses>
@@
 <pinref part="C1" gate="G$1" pin="2"/>
 </segment>
+<segment>
+<pinref part="R11" gate="G$1" pin="1"/>
+<wire x1="-271.78" y1="86.36" x2="-271.78" y2="81.28" width="0.1524" layer="91"/>
+<pinref part="GND37" gate="1" pin="GND"/>
+</segment>
 </net>
 <net name="+3V3" class="0">
@@
 <pinref part="C4" gate="G$1" pin="1"/>
 <pinref part="C3" gate="G$1" pin="1"/>
-<label x="-266.7" y="116.84" size="1.778" layer="95" rot="R180" xref="yes"/>
+<label x="-284.48" y="116.84" size="1.778" layer="95" rot="R180" xref="yes"/>
 <wire x1="-228.6" y1="116.84" x2="-254" y2="116.84" width="0.1524" layer="91"/>
 <wire x1="-254" y1="116.84" x2="-261.62" y2="116.84" width="0.1524" layer="91"/>
-<wire x1="-261.62" y1="116.84" x2="-266.7" y2="116.84" width="0.1524" layer="91"/>
+<wire x1="-261.62" y1="116.84" x2="-271.78" y2="116.84" width="0.1524" layer="91"/>
+<wire x1="-271.78" y1="116.84" x2="-284.48" y2="116.84" width="0.1524" layer="91"/>
 <wire x1="-261.62" y1="114.3" x2="-261.62" y2="116.84" width="0.1524" layer="91"/>
 <junction x="-261.62" y="116.84"/>
 <wire x1="-254" y1="114.3" x2="-254" y2="116.84" width="0.1524" layer="91"/>
 <junction x="-254" y="116.84"/>
+<pinref part="R10" gate="G$1" pin="2"/>
+<wire x1="-271.78" y1="111.76" x2="-271.78" y2="116.84" width="0.1524" layer="91"/>
+<junction x="-271.78" y="116.84"/>
 </segment>
 <segment>
@@
 </segment>
 </net>
+<net name="N$1" class="0">
+<segment>
+<pinref part="R11" gate="G$1" pin="2"/>
+<pinref part="R10" gate="G$1" pin="1"/>
+<wire x1="-271.78" y1="96.52" x2="-271.78" y2="101.6" width="0.1524" layer="91"/>
+</segment>
+</net>

Commit message: PCB
Connections:
- net +5V: now also C1.1, D2.IN, U$1.2, U2.BIAS
- net OUT: no longer C1.1, D2.IN, U$1.2, U2.BIAS
Changed lines of the file:
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@@
 <part name="R11" library="rcl" library_urn="urn:adsk.eagle:library:334" deviceset="R-US_" device="R0805" package3d_urn="urn:adsk.eagle:package:23553/2" value="??"/>
 <part name="GND37" library="supply1" library_urn="urn:adsk.eagle:library:371" deviceset="GND" device=""/>
+<part name="P+1" library="supply1" library_urn="urn:adsk.eagle:library:371" deviceset="+5V" device=""/>
 </parts>
 <sheets>
@@
 <instance part="GND37" gate="1" x="-271.78" y="78.74" smashed="yes">
 <attribute name="VALUE" x="-274.32" y="76.2" size="1.778" layer="96"/>
+</instance>
+<instance part="P+1" gate="1" x="-88.9" y="116.84" smashed="yes" rot="R270">
+<attribute name="VALUE" x="-93.98" y="119.38" size="1.778" layer="96"/>
 </instance>
 </instances>
@@
 <pinref part="P+3" gate="1" pin="+5V"/>
 </segment>
+<segment>
+<pinref part="U2" gate="A" pin="BIAS"/>
+<wire x1="-147.32" y1="109.22" x2="-139.7" y2="109.22" width="0.1524" layer="91"/>
+<wire x1="-139.7" y1="106.68" x2="-139.7" y2="109.22" width="0.1524" layer="91"/>
+<wire x1="-139.7" y1="106.68" x2="-144.78" y2="106.68" width="0.1524" layer="91"/>
+<label x="-144.78" y="106.68" size="1.778" layer="95" rot="R180" xref="yes"/>
+<wire x1="-139.7" y1="109.22" x2="-101.6" y2="109.22" width="0.1524" layer="91"/>
+<wire x1="-101.6" y1="109.22" x2="-101.6" y2="104.14" width="0.1524" layer="91"/>
+<junction x="-139.7" y="109.22"/>
+<pinref part="D2" gate="G$1" pin="IN"/>
+<wire x1="-101.6" y1="116.84" x2="-91.44" y2="116.84" width="0.1524" layer="91"/>
+<wire x1="-109.22" y1="137.16" x2="-101.6" y2="137.16" width="0.1524" layer="91"/>
+<wire x1="-101.6" y1="137.16" x2="-101.6" y2="116.84" width="0.1524" layer="91"/>
+<junction x="-101.6" y="116.84"/>
+<wire x1="-101.6" y1="109.22" x2="-101.6" y2="116.84" width="0.1524" layer="91"/>
+<junction x="-101.6" y="109.22"/>
+<pinref part="C1" gate="G$1" pin="1"/>
+<pinref part="U$1" gate="G$1" pin="2"/>
+<pinref part="P+1" gate="1" pin="+5V"/>
+</segment>
 </net>
 <net name="SDA" class="0">
@@
 <net name="OUT" class="0">
 <segment>
-<pinref part="U2" gate="A" pin="BIAS"/>
-<wire x1="-147.32" y1="109.22" x2="-139.7" y2="109.22" width="0.1524" layer="91"/>
-<wire x1="-139.7" y1="106.68" x2="-139.7" y2="109.22" width="0.1524" layer="91"/>
-<wire x1="-139.7" y1="106.68" x2="-144.78" y2="106.68" width="0.1524" layer="91"/>
-<label x="-144.78" y="106.68" size="1.778" layer="95" rot="R180" xref="yes"/>
-<wire x1="-139.7" y1="109.22" x2="-101.6" y2="109.22" width="0.1524" layer="91"/>
-<wire x1="-101.6" y1="109.22" x2="-101.6" y2="104.14" width="0.1524" layer="91"/>
-<junction x="-139.7" y="109.22"/>
-<pinref part="D2" gate="G$1" pin="IN"/>
-<wire x1="-101.6" y1="116.84" x2="-91.44" y2="116.84" width="0.1524" layer="91"/>
-<wire x1="-109.22" y1="137.16" x2="-101.6" y2="137.16" width="0.1524" layer="91"/>
-<wire x1="-101.6" y1="137.16" x2="-101.6" y2="116.84" width="0.1524" layer="91"/>
-<junction x="-101.6" y="116.84"/>
-<label x="-91.44" y="116.84" size="1.778" layer="95" xref="yes"/>
-<wire x1="-101.6" y1="109.22" x2="-101.6" y2="116.84" width="0.1524" layer="91"/>
-<junction x="-101.6" y="109.22"/>
-<pinref part="C1" gate="G$1" pin="1"/>
-<pinref part="U$1" gate="G$1" pin="2"/>
-</segment>
-<segment>
 <pinref part="U2" gate="A" pin="FB/SENSE"/>

Commit message: PCB
Connections:
- removed net OUT: U2.FB/SENSE
- net +5V: now also U2.FB/SENSE
Changed lines of the file:
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@@
 <part name="GND37" library="supply1" library_urn="urn:adsk.eagle:library:371" deviceset="GND" device=""/>
 <part name="P+1" library="supply1" library_urn="urn:adsk.eagle:library:371" deviceset="+5V" device=""/>
+<part name="P+4" library="supply1" library_urn="urn:adsk.eagle:library:371" deviceset="+5V" device=""/>
 </parts>
 <sheets>
@@
 <instance part="P+1" gate="1" x="-88.9" y="116.84" smashed="yes" rot="R270">
 <attribute name="VALUE" x="-93.98" y="119.38" size="1.778" layer="96"/>
+</instance>
+<instance part="P+4" gate="1" x="-238.76" y="111.76" smashed="yes" rot="R90">
+<attribute name="VALUE" x="-233.68" y="109.22" size="1.778" layer="96" rot="R180"/>
 </instance>
 </instances>
@@
 <pinref part="P+1" gate="1" pin="+5V"/>
 </segment>
+<segment>
+<pinref part="U2" gate="A" pin="FB/SENSE"/>
+<wire x1="-228.6" y1="111.76" x2="-236.22" y2="111.76" width="0.1524" layer="91"/>
+<pinref part="P+4" gate="1" pin="+5V"/>
+</segment>
 </net>
 <net name="SDA" class="0">
@@
 </segment>
 </net>
-<net name="OUT" class="0">
-<segment>
-<pinref part="U2" gate="A" pin="FB/SENSE"/>
-<wire x1="-228.6" y1="111.76" x2="-236.22" y2="111.76" width="0.1524" layer="91"/>
-<label x="-236.22" y="111.76" size="1.778" layer="95" rot="R180" xref="yes"/>
-</segment>
-</net>
