File: PCB/CertStack/CertStack.sch (EAGLE design)
At the start: 49 parts, among them J1 MEM2075-00-140-01-A, Q1 SI2302, Q2 SI2302, Q3 SI2302, Q4 SI2302, Q5 MMBT2222A, T1 DMP3098L-7, U1 TEENSY-32, U2 LT1374CS8-5PBF, U3 SST26VF064B-104V/MN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

Commit message: linear reg
Parts:
- added C13, C16, C18: 1uF, rcl:C-USC0805
- added C14, C15: 10uF, rcl:C-USC0805
- added U6: ADP7158ACPZ-3.3-R7, ADP7158ACPZ-3.3-R7:ADP7158ACPZ-3.3-R7
Connections:
- new net N$4: C13.2, U6.BYP
- new net N$5: C16.1, U6.VREG
- new net N$8: C18.1, U6.REF, U6.REF_SENSE
- net +3V3: now also C15.1, U6.VOUT, U6.VOUT-1, U6.VOUT_SENSE
- net +5V: now also C14.1, U6.EN, U6.VIN, U6.VIN-1
- net GND: now also C13.1, C14.2, C15.2, C16.2, C18.2
Other:
- moved on the sheet: R5

Commit message: PCB
Parts:
- removed C16, C18: 1uF, rcl:C-USC0805
- added IMU1: MLX90395KDCMLX90395, MLX90395KDC:MLX90395KDCMLX90395
- C13: value 1uF -> 4.7uF
- C14: device rcl:C-USC0805 -> SparkFun-Capacitors:10UF-1206-6.3V-20%
- C15: value 10uF -> 100nF
- U6: value ADP7158ACPZ-3.3-R7 -> ZLDO1117G33TA; device ADP7158ACPZ-3.3-R7:ADP7158ACPZ-3.3-R7 -> ZLDO1117G33TA:ZLDO1117G33TA
Connections:
- removed net N$5: C16.1, U6.VREG
- removed net N$8: C18.1, U6.REF, U6.REF_SENSE
- net +3V3: now also C13.2, IMU1./CS, IMU1.A0, IMU1.VDD; no longer U6.VOUT-1, U6.VOUT_SENSE
- net +5V: no longer U6.EN, U6.VIN-1
- net GND: now also IMU1.MISO, IMU1.VSS, U6.GND; no longer C16.2, C18.2
- net N$4: now also IMU1.INT; no longer C13.2, U6.BYP
- net SCL: now also IMU1.SCK
- net SDA: now also IMU1.SDA
Other:
- moved on the sheet: C13, C14, C15

Commit message: PCB
Parts:
- added C16, C17: (no value), rcl:C-USC0805
- added L1: IHLP3232DZER6R8M11, mylibrary:IHLP3232DZER6R8M11
- U$1: value IHLP3232DZER6R8M11 -> KIONIX_KXTJ3-1057; device mylibrary:IHLP3232DZER6R8M11 -> KIONIX_KXTJ3-1057:KIONIX_KXTJ3-1057
Connections:
- net +3V3: now also C16.1, C17.1, U$1.IO_VDD, U$1.VDD; no longer U1.3V3-1
- net +5V: now also L1.2; no longer U$1.2
- net GND: now also C16.2, C17.2, U$1.GND1, U$1.GND2
- net SCL: now also U$1.SCLK/SCL
- net SDA: now also U$1.SDI-SDA
- net VSW: now also L1.1; no longer U$1.1
Changed lines of the file:
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@@
 <?xml version="1.0" encoding="utf-8"?>
 <!DOCTYPE eagle SYSTEM "eagle.dtd">
-<eagle version="9.5.2">
+<eagle version="9.6.1">
 <drawing>
 <settings>
-<setting alwaysvectorfont="no"/>
+<setting alwaysvectorfont="yes"/>
 <setting verticaltext="up"/>
 </settings>
@@
 <part name="P+8" library="supply1" library_urn="urn:adsk.eagle:library:371" deviceset="+5V" device=""/>
 <part name="R5" library="rcl" library_urn="urn:adsk.eagle:library:334" deviceset="R-US_" device="R0805" package3d_urn="urn:adsk.eagle:package:23553/2" value="100"/>
-<part name="+3V8" library="supply1" library_urn="urn:adsk.eagle:library:371" deviceset="+3V3" device=""/>
 <part name="GND3" library="supply1" library_urn="urn:adsk.eagle:library:371" deviceset="GND" device=""/>
 <part name="Q1" library="SI2302" deviceset="SI2302" device=""/>
@@
 <part name="D1" library="PMEG4020ETP_115" deviceset="PMEG4020ETP,115" device=""/>
 <part name="C1" library="T491X106K050AT" deviceset="T491X106K050AT" device=""/>
-<part name="U$1" library="mylibrary" deviceset="IHLP3232DZER6R8M11" device=""/>
+<part name="L1" library="mylibrary" deviceset="IHLP3232DZER6R8M11" device=""/>
 <part name="R10" library="rcl" library_urn="urn:adsk.eagle:library:334" deviceset="R-US_" device="R0805" package3d_urn="urn:adsk.eagle:package:23553/2" value="??"/>
 <part name="R11" library="rcl" library_urn="urn:adsk.eagle:library:334" deviceset="R-US_" device="R0805" package3d_urn="urn:adsk.eagle:package:23553/2" value="??"/>
@@
 <part name="+3V14" library="supply1" library_urn="urn:adsk.eagle:library:371" deviceset="+3V3" device=""/>
 <part name="C15" library="rcl" library_urn="urn:adsk.eagle:library:334" deviceset="C-US" device="C0805" package3d_urn="urn:adsk.eagle:package:23617/2" value="100nF"/>
+<part name="U$1" library="KIONIX_KXTJ3-1057" deviceset="KIONIX_KXTJ3-1057" device=""/>
+<part name="GND43" library="supply1" library_urn="urn:adsk.eagle:library:371" deviceset="GND" device=""/>
+<part name="+3V16" library="supply1" library_urn="urn:adsk.eagle:library:371" deviceset="+3V3" device=""/>
+<part name="+3V17" library="supply1" library_urn="urn:adsk.eagle:library:371" deviceset="+3V3" device=""/>
+<part name="C16" library="rcl" library_urn="urn:adsk.eagle:library:334" deviceset="C-US" device="C0805" package3d_urn="urn:adsk.eagle:package:23617/2"/>
+<part name="C17" library="rcl" library_urn="urn:adsk.eagle:library:334" deviceset="C-US" device="C0805" package3d_urn="urn:adsk.eagle:package:23617/2"/>
+<part name="GND44" library="supply1" library_urn="urn:adsk.eagle:library:371" deviceset="GND" device=""/>
 </parts>
 <sheets>
@@
 <attribute name="VALUE" x="-319.278" y="97.79" size="1.778" layer="96" rot="R90"/>
 </instance>
-<instance part="+3V8" gate="G$1" x="-355.6" y="35.56" smashed="yes">
-<attribute name="VALUE" x="-353.06" y="35.56" size="1.778" layer="96" rot="R90"/>
-</instance>
 <instance part="GND3" gate="1" x="-411.48" y="40.64" smashed="yes" rot="R270">
 <attribute name="VALUE" x="-414.02" y="43.18" size="1.778" layer="96" rot="R270"/>
@@
 <attribute name="NAME" x="-105.41" y="99.06" size="1.778" layer="95" rot="R90"/>
 </instance>
-<instance part="U$1" gate="G$1" x="-114.3" y="116.84" smashed="yes"/>
+<instance part="L1" gate="G$1" x="-114.3" y="116.84" smashed="yes"/>
 <instance part="R10" gate="G$1" x="-271.78" y="106.68" smashed="yes" rot="R90">
 <attribute name="NAME" x="-273.2786" y="102.87" size="1.778" layer="95" rot="R90"/>
@@
 <attribute name="NAME" x="-270.764" y="-75.565" size="1.778" layer="95"/>
 <attribute name="VALUE" x="-270.764" y="-80.391" size="1.778" layer="96"/>
+</instance>
+<instance part="U$1" gate="G$1" x="-147.32" y="-73.66" smashed="yes"/>
+<instance part="GND43" gate="1" x="-114.3" y="-73.66" smashed="yes">
+<attribute name="VALUE" x="-116.84" y="-76.2" size="1.778" layer="96"/>
+</instance>
+<instance part="+3V16" gate="G$1" x="-106.68" y="-55.88" smashed="yes" rot="R270">
+<attribute name="VALUE" x="-111.76" y="-53.34" size="1.778" layer="96"/>
+</instance>
+<instance part="+3V17" gate="G$1" x="-185.42" y="-71.12" smashed="yes" rot="R90">
+<attribute name="VALUE" x="-180.34" y="-73.66" size="1.778" layer="96" rot="R180"/>
+</instance>
+<instance part="C16" gate="G$1" x="-114.3" y="-60.96" smashed="yes">
+<attribute name="NAME" x="-113.284" y="-60.325" size="1.778" layer="95"/>
+<attribute name="VALUE" x="-113.284" y="-65.151" size="1.778" layer="96"/>
+</instance>
+<instance part="C17" gate="G$1" x="-175.26" y="-76.2" smashed="yes">
+<attribute name="NAME" x="-174.244" y="-75.565" size="1.778" layer="95"/>
+<attribute name="VALUE" x="-174.244" y="-80.391" size="1.778" layer="96"/>
+</instance>
+<instance part="GND44" gate="1" x="-175.26" y="-86.36" smashed="yes">
+<attribute name="VALUE" x="-177.8" y="-88.9" size="1.778" layer="96"/>
 </instance>
 </instances>
@@
 <junction x="-271.78" y="-81.28"/>
 </segment>
+<segment>
+<pinref part="U$1" gate="G$1" pin="GND1"/>
+<pinref part="GND43" gate="1" pin="GND"/>
+<wire x1="-129.54" y1="-66.04" x2="-114.3" y2="-66.04" width="0.1524" layer="91"/>
+<wire x1="-114.3" y1="-66.04" x2="-114.3" y2="-71.12" width="0.1524" layer="91"/>
+<pinref part="U$1" gate="G$1" pin="GND2"/>
+<wire x1="-129.54" y1="-71.12" x2="-114.3" y2="-71.12" width="0.1524" layer="91"/>
+<junction x="-114.3" y="-71.12"/>
+<pinref part="C16" gate="G$1" pin="2"/>
+<junction x="-114.3" y="-66.04"/>
+</segment>
+<segment>
+<pinref part="GND44" gate="1" pin="GND"/>
+<pinref part="C17" gate="G$1" pin="2"/>
+<wire x1="-175.26" y1="-83.82" x2="-175.26" y2="-81.28" width="0.1524" layer="91"/>
+</segment>
 </net>
 <net name="+3V3" class="0">
@@
 </segment>
 <segment>
-<pinref part="U1" gate="G$1" pin="3V3-1"/>
-<pinref part="+3V8" gate="G$1" pin="+3V3"/>
-<wire x1="-363.22" y1="30.48" x2="-355.6" y2="30.48" width="0.1524" layer="91"/>
-<wire x1="-355.6" y1="30.48" x2="-355.6" y2="33.02" width="0.1524" layer="91"/>
-</segment>
-<segment>
 <pinref part="+3V9" gate="G$1" pin="+3V3"/>
 <pinref part="POWER" gate="G$1" pin="2"/>
@@
 <junction x="-261.62" y="-73.66"/>
 </segment>
+<segment>
+<pinref part="+3V16" gate="G$1" pin="+3V3"/>
+<pinref part="U$1" gate="G$1" pin="VDD"/>
+<wire x1="-109.22" y1="-55.88" x2="-114.3" y2="-55.88" width="0.1524" layer="91"/>
+<pinref part="C16" gate="G$1" pin="1"/>
+<wire x1="-114.3" y1="-55.88" x2="-114.3" y2="-58.42" width="0.1524" layer="91"/>
+<wire x1="-129.54" y1="-60.96" x2="-121.92" y2="-60.96" width="0.1524" layer="91"/>
+<wire x1="-121.92" y1="-60.96" x2="-121.92" y2="-55.88" width="0.1524" layer="91"/>
+<wire x1="-121.92" y1="-55.88" x2="-114.3" y2="-55.88" width="0.1524" layer="91"/>
+<junction x="-114.3" y="-55.88"/>
+</segment>
+<segment>
+<pinref part="+3V17" gate="G$1" pin="+3V3"/>
+<pinref part="U$1" gate="G$1" pin="IO_VDD"/>
+<pinref part="C17" gate="G$1" pin="1"/>
+<wire x1="-165.1" y1="-71.12" x2="-175.26" y2="-71.12" width="0.1524" layer="91"/>
+<wire x1="-175.26" y1="-71.12" x2="-182.88" y2="-71.12" width="0.1524" layer="91"/>
+<wire x1="-175.26" y1="-73.66" x2="-175.26" y2="-71.12" width="0.1524" layer="91"/>
+<junction x="-175.26" y="-71.12"/>
+</segment>
 </net>
 <net name="CS_BAR" class="0">
@@
 <pinref part="IMU1" gate="G$1" pin="SCK"/>
 <wire x1="-307.34" y1="-68.58" x2="-314.96" y2="-68.58" width="0.1524" layer="91"/>
+</segment>
+<segment>
+<pinref part="U$1" gate="G$1" pin="SCLK/SCL"/>
+<wire x1="-129.54" y1="-86.36" x2="-119.38" y2="-86.36" width="0.1524" layer="91"/>
+<label x="-119.38" y="-86.36" size="1.778" layer="95" xref="yes"/>
 </segment>
 </net>
@@
 <junction x="-101.6" y="109.22"/>
 <pinref part="C1" gate="G$1" pin="1"/>
-<pinref part="U$1" gate="G$1" pin="2"/>
+<pinref part="L1" gate="G$1" pin="2"/>
 <pinref part="P+1" gate="1" pin="+5V"/>
 </segment>
@@
 <pinref part="IMU1" gate="G$1" pin="SDA"/>
 <wire x1="-307.34" y1="-73.66" x2="-314.96" y2="-73.66" width="0.1524" layer="91"/>
+</segment>
+<segment>
+<pinref part="U$1" gate="G$1" pin="SDI-SDA"/>
+<wire x1="-165.1" y1="-66.04" x2="-172.72" y2="-66.04" width="0.1524" layer="91"/>
+<label x="-172.72" y="-66.04" size="1.778" layer="95" rot="R180" xref="yes"/>
 </segment>
 </net>
@@
 <pinref part="D1" gate="G$1" pin="K"/>
 <wire x1="-127" y1="104.14" x2="-127" y2="116.84" width="0.1524" layer="91"/>
-<pinref part="U$1" gate="G$1" pin="1"/>
-</segment>
-</net>
+<pinref part="L1" gate="G$1" pin="1"/>
+</segment>
+</net>

Commit message: PCB:
Parts:
- C16, C17: value (none) -> 0.1uF
Connections:
- net +3V3: now also U$1.CS
- net GND: now also U$1.NC, U$1.SDO-ADDR, U$1.TRIG
Changed lines of the file:
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@@
 <?xml version="1.0" encoding="utf-8"?>
 <!DOCTYPE eagle SYSTEM "eagle.dtd">
-<eagle version="9.6.1">
+<eagle version="9.5.2">
 <drawing>
 <settings>
-<setting alwaysvectorfont="yes"/>
+<setting alwaysvectorfont="no"/>
 <setting verticaltext="up"/>
 </settings>
@@
 <part name="+3V16" library="supply1" library_urn="urn:adsk.eagle:library:371" deviceset="+3V3" device=""/>
 <part name="+3V17" library="supply1" library_urn="urn:adsk.eagle:library:371" deviceset="+3V3" device=""/>
-<part name="C16" library="rcl" library_urn="urn:adsk.eagle:library:334" deviceset="C-US" device="C0805" package3d_urn="urn:adsk.eagle:package:23617/2"/>
-<part name="C17" library="rcl" library_urn="urn:adsk.eagle:library:334" deviceset="C-US" device="C0805" package3d_urn="urn:adsk.eagle:package:23617/2"/>
+<part name="C16" library="rcl" library_urn="urn:adsk.eagle:library:334" deviceset="C-US" device="C0805" package3d_urn="urn:adsk.eagle:package:23617/2" value="0.1uF"/>
+<part name="C17" library="rcl" library_urn="urn:adsk.eagle:library:334" deviceset="C-US" device="C0805" package3d_urn="urn:adsk.eagle:package:23617/2" value="0.1uF"/>
 <part name="GND44" library="supply1" library_urn="urn:adsk.eagle:library:371" deviceset="GND" device=""/>
+<part name="GND45" library="supply1" library_urn="urn:adsk.eagle:library:371" deviceset="GND" device=""/>
+<part name="GND46" library="supply1" library_urn="urn:adsk.eagle:library:371" deviceset="GND" device=""/>
+<part name="+3V8" library="supply1" library_urn="urn:adsk.eagle:library:371" deviceset="+3V3" device=""/>
+<part name="GND47" library="supply1" library_urn="urn:adsk.eagle:library:371" deviceset="GND" device=""/>
 </parts>
 <sheets>
@@
 <instance part="GND44" gate="1" x="-175.26" y="-86.36" smashed="yes">
 <attribute name="VALUE" x="-177.8" y="-88.9" size="1.778" layer="96"/>
+</instance>
+<instance part="GND45" gate="1" x="-172.72" y="-60.96" smashed="yes" rot="R270">
+<attribute name="VALUE" x="-175.26" y="-58.42" size="1.778" layer="96" rot="R270"/>
+</instance>
+<instance part="GND46" gate="1" x="-167.64" y="-76.2" smashed="yes" rot="R270">
+<attribute name="VALUE" x="-170.18" y="-73.66" size="1.778" layer="96" rot="R270"/>
+</instance>
+<instance part="+3V8" gate="G$1" x="-121.92" y="-76.2" smashed="yes" rot="R270">
+<attribute name="VALUE" x="-127" y="-73.66" size="1.778" layer="96"/>
+</instance>
+<instance part="GND47" gate="1" x="-127" y="-81.28" smashed="yes" rot="R90">
+<attribute name="VALUE" x="-124.46" y="-83.82" size="1.778" layer="96" rot="R90"/>
 </instance>
 </instances>
@@
 <wire x1="-175.26" y1="-83.82" x2="-175.26" y2="-81.28" width="0.1524" layer="91"/>
 </segment>
+<segment>
+<pinref part="GND45" gate="1" pin="GND"/>
+<pinref part="U$1" gate="G$1" pin="SDO-ADDR"/>
+<wire x1="-170.18" y1="-60.96" x2="-165.1" y2="-60.96" width="0.1524" layer="91"/>
+</segment>
+<segment>
+<pinref part="U$1" gate="G$1" pin="TRIG"/>
+<pinref part="GND46" gate="1" pin="GND"/>
+</segment>
+<segment>
+<pinref part="U$1" gate="G$1" pin="NC"/>
+<pinref part="GND47" gate="1" pin="GND"/>
+</segment>
 </net>
 <net name="+3V3" class="0">
@@
 <junction x="-175.26" y="-71.12"/>
 </segment>
+<segment>
+<pinref part="U$1" gate="G$1" pin="CS"/>
+<wire x1="-129.54" y1="-76.2" x2="-124.46" y2="-76.2" width="0.1524" layer="91"/>
+<pinref part="+3V8" gate="G$1" pin="+3V3"/>
+</segment>
 </net>

Commit message: PCB
Connections:
- removed net CS_ACCEL: U1.15
- net CS_BAR: now also U1.16
- net CS_IMU: now also U1.15
Changed lines of the file:
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@@
 <label x="-228.6" y="50.8" size="1.778" layer="95" xref="yes"/>
+</segment>
+<segment>
+<pinref part="U1" gate="G$1" pin="16"/>
+<wire x1="-363.22" y1="-10.16" x2="-350.52" y2="-10.16" width="0.1524" layer="91"/>
+<label x="-350.52" y="-10.16" size="1.778" layer="95"/>
 </segment>
 </net>
@@
 <wire x1="-146.05" y1="45.72" x2="-186.69" y2="45.72" width="0.1524" layer="91"/>
 <label x="-186.69" y="45.72" size="1.778" layer="95" rot="MR0" xref="yes"/>
+</segment>
+<segment>
+<pinref part="U1" gate="G$1" pin="15"/>
+<wire x1="-363.22" y1="-15.24" x2="-350.52" y2="-15.24" width="0.1524" layer="91"/>
+<label x="-350.52" y="-15.24" size="1.778" layer="95" xref="yes"/>
 </segment>
 </net>
@@
 </segment>
 </net>
-<net name="CS_ACCEL" class="0">
-<segment>
-<pinref part="U1" gate="G$1" pin="15"/>
-<wire x1="-363.22" y1="-15.24" x2="-350.52" y2="-15.24" width="0.1524" layer="91"/>
-<label x="-350.52" y="-15.24" size="1.778" layer="95" xref="yes"/>
-</segment>
-</net>

Commit message: PCB
Parts:
- R1: value 150 -> 62
- R3: value 15 -> 71.5
Connections:
- removed net N$1: R10.1, R11.2
- new net BAT-SENSE: R10.1, R11.2, U1.23
Other:
- moved on the sheet: C1, C13, C14, C2, C3, C4, C5, CAMERA, D1, DATA, GPS, POWER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

Commit message: PCB
Parts:
- added R12, R13: 4.7k, rcl:R-US_R0805
Connections:
- net +3V3: now also R12.2, R13.2
- net SCL: now also R12.1
- net SDA: now also R13.1
Changed lines of the file:
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@@
 <?xml version="1.0" encoding="utf-8"?>
 <!DOCTYPE eagle SYSTEM "eagle.dtd">
-<eagle version="9.6.1">
+<eagle version="9.5.1">
 <drawing>
 <settings>
-<setting alwaysvectorfont="yes"/>
+<setting alwaysvectorfont="no"/>
 <setting verticaltext="up"/>
 </settings>
@@
 <part name="+3V8" library="supply1" library_urn="urn:adsk.eagle:library:371" deviceset="+3V3" device=""/>
 <part name="GND47" library="supply1" library_urn="urn:adsk.eagle:library:371" deviceset="GND" device=""/>
+<part name="R12" library="rcl" library_urn="urn:adsk.eagle:library:334" deviceset="R-US_" device="R0805" package3d_urn="urn:adsk.eagle:package:23553/2" value="4.7k"/>
+<part name="R13" library="rcl" library_urn="urn:adsk.eagle:library:334" deviceset="R-US_" device="R0805" package3d_urn="urn:adsk.eagle:package:23553/2" value="4.7k"/>
+<part name="+3V18" library="supply1" library_urn="urn:adsk.eagle:library:371" deviceset="+3V3" device=""/>
 </parts>
 <sheets>
@@
 <instance part="GND47" gate="1" x="-127" y="-81.28" smashed="yes" rot="R90">
 <attribute name="VALUE" x="-124.46" y="-83.82" size="1.778" layer="96" rot="R90"/>
+</instance>
+<instance part="R12" gate="G$1" x="-330.2" y="12.7" smashed="yes" rot="R90">
+<attribute name="NAME" x="-331.6986" y="8.89" size="1.778" layer="95" rot="R90"/>
+<attribute name="VALUE" x="-326.898" y="8.89" size="1.778" layer="96" rot="R90"/>
+</instance>
+<instance part="R13" gate="G$1" x="-320.04" y="12.7" smashed="yes" rot="R90">
+<attribute name="NAME" x="-321.5386" y="8.89" size="1.778" layer="95" rot="R90"/>
+<attribute name="VALUE" x="-316.738" y="8.89" size="1.778" layer="96" rot="R90"/>
+</instance>
+<instance part="+3V18" gate="G$1" x="-325.12" y="22.86" smashed="yes">
+<attribute name="VALUE" x="-327.66" y="17.78" size="1.778" layer="96" rot="R90"/>
 </instance>
 </instances>
@@
 <pinref part="+3V8" gate="G$1" pin="+3V3"/>
 </segment>
+<segment>
+<pinref part="R12" gate="G$1" pin="2"/>
+<pinref part="R13" gate="G$1" pin="2"/>
+<wire x1="-330.2" y1="17.78" x2="-325.12" y2="17.78" width="0.1524" layer="91"/>
+<pinref part="+3V18" gate="G$1" pin="+3V3"/>
+<wire x1="-325.12" y1="17.78" x2="-320.04" y2="17.78" width="0.1524" layer="91"/>
+<wire x1="-325.12" y1="20.32" x2="-325.12" y2="17.78" width="0.1524" layer="91"/>
+<junction x="-325.12" y="17.78"/>
+</segment>
 </net>
 <net name="CS_BAR" class="0">
@@
 <segment>
 <pinref part="U1" gate="G$1" pin="19"/>
-<wire x1="-363.22" y1="5.08" x2="-350.52" y2="5.08" width="0.1524" layer="91"/>
-<label x="-350.52" y="5.08" size="1.778" layer="95" xref="yes"/>
+<wire x1="-363.22" y1="5.08" x2="-330.2" y2="5.08" width="0.1524" layer="91"/>
+<label x="-312.42" y="5.08" size="1.778" layer="95" xref="yes"/>
 <label x="-314.96" y="-68.58" size="1.778" layer="95" rot="R180" xref="yes"/>
+<pinref part="R12" gate="G$1" pin="1"/>
+<wire x1="-330.2" y1="5.08" x2="-312.42" y2="5.08" width="0.1524" layer="91"/>
+<wire x1="-330.2" y1="7.62" x2="-330.2" y2="5.08" width="0.1524" layer="91"/>
+<junction x="-330.2" y="5.08"/>
 </segment>
 <segment>
@@
 <segment>
 <pinref part="U1" gate="G$1" pin="18"/>
-<wire x1="-363.22" y1="0" x2="-350.52" y2="0" width="0.1524" layer="91"/>
-<label x="-350.52" y="0" size="1.778" layer="95" xref="yes"/>
+<wire x1="-363.22" y1="0" x2="-320.04" y2="0" width="0.1524" layer="91"/>
+<label x="-312.42" y="0" size="1.778" layer="95" xref="yes"/>
 <label x="-314.96" y="-73.66" size="1.778" layer="95" rot="R180" xref="yes"/>
-</segment>
-<segment>
+<pinref part="R13" gate="G$1" pin="1"/>
+<wire x1="-320.04" y1="0" x2="-312.42" y2="0" width="0.1524" layer="91"/>
+<wire x1="-320.04" y1="7.62" x2="-320.04" y2="0" width="0.1524" layer="91"/>
+<junction x="-320.04" y="0"/>
+</segment>
+<segment>

Commit message: PCB
Parts:
- removed DATA: (no value), mylibrary:JST-PH-6
- added EXTN.: (no value), mylibrary:JST-PH-6
- R10: value ?? -> 30.1k
- R11: value ?? -> 10k
Connections:
- removed net CANH: DATA.6
- removed net CANL: DATA.5
- net +3V3: now also EXTN..2; no longer DATA.2
- net FET3: now also EXTN..5
- net FET4: now also EXTN..6
- net GND: now also EXTN..1; no longer DATA.1
- net SCL: now also EXTN..3; no longer DATA.3
- net SDA: now also EXTN..4; no longer DATA.4
Other:
- note added: "Magnetometer"
- moved on the sheet: C15, C16, C17, C6, CAMERA, GPS, IMU1, J1, LED1, LED2, LED3, POWER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
